File: v0.1/MCU.kicad_sch (KiCad schematic)
At the start: 1 part, among them U10 STM32U5G9ZJTxQ

Commit message: [HW] [PCB] phase #2
Connections:
- net MCO: now reaches U10.102 (PA8)
- net SWDIO: now reaches U10.107 (PA13)
- net SWCLK: now reaches U10.111 (PA14)
- net NRST: now reaches U10.134 (PB4)
- net OSC_IN: now reaches U10.26 (PH0)
- net OSC_OUT: now reaches U10.27 (PH1)
- net OSC_32IN: now reaches U10.8 (PC14)
- net OSC_32OUT: now reaches U10.9 (PC15)
