File: v0.1/v0.1.kicad_pcb (KiCad board)
At the start: 2 copper layers, 111.2 x 86.9 mm, 88 parts, among them U1 XC6206P152MR, U10 STM32U5G9ZJTxQ, U2 XC6206P282MR, U3 SY8088AAC, U4 XC6206P282MR, U9 MX66LM1G45G

Commit message: [HW] [PCB] phase #2
Parts:
- added JP10: SolderJumper_2_Open, Jumper:SolderJumper-2_P1.3mm_Open_TrianglePad1.0x1.5mm, F.Cu at (92.6, 92.8)
- added JP11: SolderJumper_2_Open, Jumper:SolderJumper-2_P1.3mm_Open_TrianglePad1.0x1.5mm, F.Cu at (92.6, 96.3)
- added JP8: SolderJumper_2_Open, Jumper:SolderJumper-2_P1.3mm_Open_TrianglePad1.0x1.5mm, F.Cu at (109.9, 94.5)
- added JP9: SolderJumper_2_Open, Jumper:SolderJumper-2_P1.3mm_Open_TrianglePad1.0x1.5mm, F.Cu at (109.9, 98.1)
- added R15: 33R, Resistor_SMD:R_0603_1608Metric, F.Cu at (99.8, 98.2)
- added R16: 4.7k, Resistor_SMD:R_0603_1608Metric, F.Cu at (118.8, 88.0)
- added R17: 4.7k, Resistor_SMD:R_0603_1608Metric, F.Cu at (118.8, 90.5)
- added R18: 10k, Resistor_SMD:R_0603_1608Metric, F.Cu at (118.8, 93.0)
- added TP13: TestPoint, TestPoint:TestPoint_Pad_D1.0mm, F.Cu at (98.1, 105.2)
- added U11: ~, Grinreflex:FPC-SMD_24P-P0.50_SHOU-HAN_CTSJ-H2.0, B.Cu at (109.9, 75.8)
- moved C17 38.9 mm to (83.1, 113.0)
- moved Q1 38.9 mm to (79.4, 112.8)
- moved R7 38.9 mm to (78.2, 117.2)
- moved R8 38.9 mm to (80.7, 117.2)
- moved R9 38.9 mm to (83.3, 117.2)
- moved U6 38.9 mm to (72.0, 112.4)
Connections:
- net /MCU/DCMI_D6 renamed /Camera/DVP_D6
- net /MCU/DCMI_D7 renamed /Camera/DVP_D7
- JP1 pad 1: unconnected-(JP1-A-Pad1) -> /2v8
- JP2 pad 1: unconnected-(JP2-A-Pad1) -> /DVDD-1v5
- JP3 pad 1: unconnected-(JP3-A-Pad1) -> /AVDD-2v8
- JP4 pad 1: unconnected-(JP4-A-Pad1) -> /AF-2v8
- JP6 pad 1: unconnected-(JP6-A-Pad1) -> /+5V
- TP4 pad 1: /FLASH/RESET -> /RESET
- U10 pad 100: /MCU/DCMI_D2 -> /Camera/DVP_D2
- U10 pad 101: /MCU/DCMI_D3 -> /Camera/DVP_D3
- U10 pad 102: unconnected-(U10-PA8-Pad102) -> /Camera/DVP_XCLK
- U10 pad 103: /MCU/DCMI_D0 -> /MCU/usart1_tx
- U10 pad 104: /MCU/DCMI_D1 -> /MCU/usart1_rx
- U10 pad 107: unconnected-(U10-PA13-Pad107) -> /MCU/SWDIO
- U10 pad 111: unconnected-(U10-PA14-Pad111) -> /MCU/SWCLK
- U10 pad 128: unconnected-(U10-PG13-Pad128) -> /I2C1_SDA
- U10 pad 129: unconnected-(U10-PG14-Pad129) -> /I2C1_SCL
- U10 pad 134: unconnected-(U10-PB4-Pad134) -> /RESET
- U10 pad 135: unconnected-(U10-PB5-Pad135) -> /MCU/spi1_mosi
- U10 pad 136: /MCU/DCMI_D5 -> /Camera/DVP_D5
- U10 pad 26: unconnected-(U10-PH0-Pad26) -> /MCU/OSC_IN
- U10 pad 27: unconnected-(U10-PH1-Pad27) -> /MCU/OSC_OUT
- U10 pad 3: /MCU/DCMI_D4 -> /Camera/DVP_D4
- U10 pad 38: unconnected-(U10-PA2-Pad38) -> /MCU/usart2_tx
- U10 pad 39: unconnected-(U10-PA3-Pad39) -> /MCU/usart2_rx
- U10 pad 43: unconnected-(U10-PA5-Pad43) -> /MCU/spi1_sck
- U10 pad 44: /MCU/DCMI_PCLK -> /MCU/spi1_miso
- U10 pad 46: unconnected-(U10-PB0-Pad46) -> /MCU/spi1_nss
- U10 pad 8: unconnected-(U10-PC14-Pad8) -> /MCU/OSC_32IN
- U10 pad 9: unconnected-(U10-PC15-Pad9) -> /MCU/OSC_32OUT
- U10 pad 98: /MCU/DCMI_D0 -> /Camera/DVP_D0
- U10 pad 99: /MCU/DCMI_D1 -> /Camera/DVP_D1
- U6 pad 3: /LCD/LCD_RESET -> /RESET
- U9 pad 3: /FLASH/RESET -> /RESET
