File: v0.1/v0.1.kicad_pcb (KiCad board)
At the start: 4 copper layers, 66.4 x 47.2 mm, 140 parts, among them J1 Conn_01x05_Pin, J2 Conn_01x04_Pin, J3 Conn_01x02_Pin, J4 Conn_01x02_Pin, U1 XC6206P152MR, U10 STM32U5G9ZJTxQ, U2 XC6206P282MR, U3 SY8088AAC, U4 XC6206P282MR, U9 MX66LM1G45G, X1 32.768kHz, X2 16MHz

Commit message: [HW] [PCB] v0.1_Y48 revision
Parts:
- D3: footprint Diode_SMD:D_SOD-323 -> Grinreflex:SOD-523F_L1.2-W0.8-LS1.7-RD
- R19, R6, R7, TP8: moved to B.Cu
- U9: footprint Package_SO:SOP-16_3.9x9.9mm_P1.27mm -> Package_SO:SOIC-16W_7.5x10.3mm_P1.27mm
- moved J3 14.7 mm to (93.4, 49.5), turned to -90 degrees
- moved R6 7.50 mm to (115.4, 52.3), turned to 180 degrees
- moved R7 4.69 mm to (117.9, 58.8), turned to 180 degrees
- moved R19 3.16 mm to (113.7, 59.7), turned to 0 degrees
- moved TP17 2.95 mm to (121.4, 52.1)
- moved TP9 2.83 mm to (119.4, 50.1)
- moved C24 1.00 mm to (117.3, 56.1)
- moved R21 0.85 mm to (117.3, 66.8)
- moved C23 0.60 mm to (117.3, 54.4)
- moved TP10 0.20 mm to (122.9, 50.5)
- moved TP16 0.10 mm to (123.0, 53.9)
- turned TP8 to 180 degrees
Connections:
- U10 pad 134: /RESET -> unconnected-(U10-PB4-Pad134)
- U10 pad 28: unconnected-(U10-NRST-Pad28) -> /RESET
Routing:
- net /RESET: track 107.6 -> 137.2 mm, vias 5 -> 6
- net /MCU/usart1_rx: track 18.7 -> 37.2 mm, vias 0 -> 1
- net /MCU/usart1_tx: track 21.8 -> 35.0 mm, vias 0 -> 1
- net /FLASH/SI2: track 25.2 -> 35.3 mm
- net /3v3_pwr: track 136.7 -> 126.8 mm
- net /MCU/hspi1_ncs: track 16.5 -> 9.91 mm, vias 2 -> 1
- net /FLASH/SCLK: track 12.4 -> 7.67 mm, vias 0 -> 1
- net /Camera/DVP_D4: track 29.9 -> 34.3 mm
- net /FLASH/SI6: track 25.4 -> 22.3 mm
- net /MCU/hspi1_clk: track 15.3 -> 18.3 mm
- net /FLASH/DQS: track 29.1 -> 27.0 mm, vias 2 -> 0
- net /FLASH/SI4: track 28.7 -> 30.9 mm
- net /FLASH/SI5: track 27.3 -> 29.3 mm
- net /FLASH/SI0: track 30.8 -> 32.4 mm
- net /MCU/DCMI_PCLK: track 29.9 -> 31.0 mm
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
Commit message: [HW] [PCB] revision v0.1_Y49
Parts:
- removed the JP9 at (105.6, 62.0)
- removed the R17 at (103.6, 50.9)
- removed the R3 at (139.3, 55.2)
- removed the R4 at (139.3, 57.0)
- added C38: 100nf, Capacitor_SMD:C_0603_1608Metric, B.Cu at (126.4, 77.2)
- added C54: 100nf, Capacitor_SMD:C_0603_1608Metric, F.Cu at (121.1, 85.5)
- added R19: 1.5k, Resistor_SMD:R_0603_1608Metric, F.Cu at (118.0, 83.2)
- added TP19: TestPoint, TestPoint:TestPoint_Pad_D1.0mm, F.Cu at (130.7, 89.1)
- added TP20: TestPoint, TestPoint:TestPoint_Pad_D1.0mm, F.Cu at (131.8, 91.0)
- added TP21: TestPoint, TestPoint:TestPoint_Pad_D1.0mm, F.Cu at (134.1, 91.2)
- added TP22: TestPoint, TestPoint:TestPoint_Pad_D1.0mm, F.Cu at (135.2, 89.3)
- added TP23: TestPoint, TestPoint:TestPoint_Pad_D1.0mm, B.Cu at (102.4, 79.4)
- added TP24: TestPoint, TestPoint:TestPoint_Pad_D1.0mm, B.Cu at (102.4, 81.8)
- added TP25: TestPoint, TestPoint:TestPoint_Pad_D1.0mm, B.Cu at (118.0, 75.0)
- added U12: ~, Grinreflex:SOT-23-3_L2.9-W1.6-P1.90-LS2.8-BR, F.Cu at (118.5, 86.8)
- R13: renamed from R15; footprint Resistor_SMD:R_0603_1608Metric -> Resistor_SMD:R_0402_1005Metric
- R14: renamed from R16; footprint Resistor_SMD:R_0603_1608Metric -> Resistor_SMD:R_0402_1005Metric
- R18: value 200k -> 100k
- R6: renamed from R8; footprint Resistor_SMD:R_0603_1608Metric -> Resistor_SMD:R_0402_1005Metric
- R7: renamed from R9; footprint Resistor_SMD:R_0603_1608Metric -> Resistor_SMD:R_0402_1005Metric
- moved R18 34.7 mm to (119.5, 83.2), turned to 90 degrees
- moved J3 16.2 mm to (109.6, 49.8)
- moved D1 15.3 mm to (106.5, 62.8), turned to 90 degrees
- moved C33 14.0 mm to (131.4, 81.1), turned to 90 degrees
- moved C1 14.0 mm to (104.7, 62.8), turned to 90 degrees
- moved C32 13.7 mm to (126.2, 73.9)
- moved C37 12.8 mm to (140.8, 70.7), turned to 90 degrees
- moved C36 11.2 mm to (140.2, 74.0), turned to -90 degrees
- moved C34 10.3 mm to (138.6, 75.8)
- moved C35 10.1 mm to (133.2, 81.1)
- moved C30 9.83 mm to (131.3, 68.8)
- moved C29 9.57 mm to (133.2, 67.2)
- moved R7 7.30 mm to (94.2, 69.5), turned to 90 degrees
- moved R6 6.75 mm to (93.2, 70.1)
- moved D2 6.62 mm to (103.3, 70.0), turned to 90 degrees
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- renumbered C27 to C39, C28 to C40, C29 to C41, C30 to C42, C31 to C43, C32 to C44, C33 to C45, C34 to C46, C35 to C47, C36 to C48, C37 to C49, C38 to C50, C39 to C51, C40 to C52, C41 to C53, C42 to C55, JP11 to JP10, JP12 to JP11, JP13 to JP12, JP14 to JP13, JP10 to JP9, R12 to R10, R13 to R11, R14 to R12, R19 to R15, R20 to R16, R21 to R17, R5 to R3, R6 to R4, R7 to R5, R10 to R8, R11 to R9
Connections:
- net /MCU/DCMI_HS renamed /Camera/DVP_HSYNC
- net /MCU/DCMI_PCLK renamed /Camera/DVP_PCLK
- net /MCU/DCMI_VS renamed /Camera/DVP_VSYNC
- C28 pad 1: /3v3_pwr -> GND
- C28 pad 2: GND -> /3v3_pwr
- C29 pad 1: GND -> /3v3_pwr
- C29 pad 2: /3v3_pwr -> GND
- C30 pad 1: /3v3_pwr -> GND
- C30 pad 2: GND -> /3v3_pwr
- C31 pad 1: GND -> /3v3_pwr
- C31 pad 2: /3v3_pwr -> GND
- C32 pad 1: /3v3_pwr -> GND
- C32 pad 2: GND -> /3v3_pwr
- C33 pad 1: GND -> /3v3_pwr
- C33 pad 2: /3v3_pwr -> GND
- C34 pad 1: /3v3_pwr -> GND
- C34 pad 2: GND -> /3v3_pwr
- C35 pad 1: GND -> /3v3_pwr
- C35 pad 2: /3v3_pwr -> GND
- C36 pad 1: /3v3_pwr -> GND
- C36 pad 2: GND -> /3v3_pwr
- C37 pad 1: GND -> /3v3_pwr
- C37 pad 2: /3v3_pwr -> GND
- R18 pad 1: /USB-C/USBC_DETECT -> Net-(U12-RESET)
- U10 pad 1: unconnected-(U10-PE2-Pad1) -> Net-(U10-PE2)
- U10 pad 113: /MCU/DCMI_D8 -> unconnected-(U10-PC10-Pad113)
- U10 pad 116: /i2c6_sda -> unconnected-(U10-PD0-Pad116)
- U10 pad 117: /i2c6_scl -> unconnected-(U10-PD1-Pad117)
- U10 pad 119: unconnected-(U10-PD3-Pad119) -> /LCD/LCD_SDA
- U10 pad 120: unconnected-(U10-PD4-Pad120) -> /LCD/LCD_SCL
- U10 pad 2: unconnected-(U10-PE3-Pad2) -> Net-(U10-PE3)
- U10 pad 4: unconnected-(U10-PE5-Pad4) -> Net-(U10-PE5)
- U10 pad 5: unconnected-(U10-PE6-Pad5) -> Net-(U10-PE6)
- U6 pad 5: /i2c6_sda -> /LCD/LCD_SDA
- U6 pad 6: /i2c6_scl -> /LCD/LCD_SCL
- U8 pad 11: Net-(JP9-A) -> unconnected-(U8-FLT/-Pad11)
Routing:
- net /i2c6_sda: track 31.4 -> 0.00 mm, vias 2 -> 0
- net /i2c6_scl: track 30.0 -> 0.00 mm, vias 2 -> 0
- net /LCD/LCD_SDA: track 0.00 -> 29.4 mm, vias 0 -> 1
- net /LCD/LCD_SCL: track 0.00 -> 28.8 mm, vias 0 -> 1
- net GND: track 69.9 -> 52.6 mm, vias 153 -> 150
- net /Camera/DVP_VSYNC: track 27.9 -> 41.6 mm, vias 3 -> 4
- net /Camera/DVP_HSYNC: track 30.2 -> 42.5 mm, vias 3 -> 4
- net /RESET: track 137.2 -> 149.4 mm, vias 6 -> 7
- net /MCU/usart1_rx: track 37.2 -> 26.0 mm, vias 1 -> 0
- net /3v3_pwr: track 126.8 -> 116.7 mm
- net /Power/3v3: track 56.6 -> 46.6 mm
- net /MCU/usart1_tx: track 35.0 -> 26.4 mm, vias 1 -> 0
- net /+5V: track 27.0 -> 20.5 mm
- net Net-(U10-PE5): track 0.00 -> 5.15 mm
- net Net-(U10-PE3): track 0.00 -> 4.95 mm
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
Commit message: [HW] [PCB] PCB Revision 0.2_Y50; DK1
Parts:
- removed the JP3 at (93.9, 76.5)
- added J3: Conn_01x02_Pin, Connector_PinHeader_2.54mm:PinHeader_1x02_P2.54mm_Vertical, F.Cu at (142.2, 55.8)
- added R20: 100k, Resistor_SMD:R_0402_1005Metric, B.Cu at (114.9, 88.3)
- C47, C49, C50, C51, C52, C53, C54: footprint Capacitor_SMD:C_0603_1608Metric -> Capacitor_SMD:C_0402_1005Metric
- J2: value Conn_01x04_Pin -> Conn_01x02_Pin; footprint Connector_PinHeader_2.54mm:PinHeader_1x04_P2.54mm_Vertical -> Connector_PinHeader_2.54mm:PinHeader_1x02_P2.54mm_Vertical
- R1, R16, R18, R19, R2: footprint Resistor_SMD:R_0603_1608Metric -> Resistor_SMD:R_0402_1005Metric
- R10: renamed from R12; footprint Resistor_SMD:R_0603_1608Metric -> Resistor_SMD:R_0402_1005Metric
- R11: renamed from R10; footprint Resistor_SMD:R_0603_1608Metric -> Resistor_SMD:R_0402_1005Metric
- R12: renamed from R11; footprint Resistor_SMD:R_0603_1608Metric -> Resistor_SMD:R_0402_1005Metric
- R4, R5: value 27R -> 33R
- U11: footprint Grinreflex:FPC-SMD_24P-P0.50_SHOU-HAN_CTSJ-H2.0 -> Grinreflex:FFC-SMD_24P-P0.50_FH34SRJ-24S-0.5SH
- U6: footprint Grinreflex:FPC-SMD_8P-P0.50_AFC24-S08FCA-00 -> Grinreflex:FPC-SMD_8P-P0.50_FH34D-8S-0.5SH-50
- moved SW1 24.1 mm to (86.5, 78.1), turned to 90 degrees
- moved TP2 13.6 mm to (91.9, 74.2)
- moved C10 7.36 mm to (100.9, 79.8)
- moved J2 6.54 mm to (145.9, 55.8), turned to 0 degrees
- moved L1 5.32 mm to (91.6, 77.5), turned to -90 degrees
- moved J5 5.15 mm to (146.2, 63.6), turned to 0 degrees
- moved JP11 4.95 mm to (100.5, 76.5)
- moved TP24 4.07 mm to (102.8, 77.7)
- moved JP6 4.03 mm to (94.0, 76.6)
- moved TP23 3.45 mm to (105.3, 77.6)
- moved JP2 3.35 mm to (104.6, 86.0), turned to 90 degrees
- moved C2 2.95 mm to (89.0, 86.4), turned to 180 degrees
- moved TP6 2.91 mm to (104.5, 83.3)
- moved JP4 2.88 mm to (105.7, 76.5)
- moved JP5 2.75 mm to (103.0, 76.5)
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- renumbered J3 to J4, J4 to J5, JP11 to JP10, JP12 to JP11, JP13 to JP12, JP4 to JP3, JP5 to JP4, JP6 to JP5, JP7 to JP6, JP8 to JP7, JP9 to JP8, JP10 to JP9
Connections:
- C22 pad 1: Net-(D5-A) -> Net-(D5-K)
- D5 pad 1: /USB-C/VBUS -> Net-(D5-K)
- D5 pad 2: Net-(D5-A) -> /USB-C/VBUS
- J2 pad 1: /MCU/spi1_sck -> /MCU/spi1_mosi
- J2 pad 2: /MCU/spi1_nss -> /MCU/spi1_miso
- U10 pad 119: /LCD/LCD_SDA -> /LCD/LCD_SCL
- U10 pad 120: /LCD/LCD_SCL -> /LCD/LCD_SDA
- U8 pad 8: Net-(D5-A) -> Net-(D5-K)
Routing:
- net /RESET: track 149.4 -> 168.8 mm, vias 7 -> 6
- net GND: track 52.6 -> 33.3 mm, vias 150 -> 162
- net /MCU/spi1_sck: track 9.96 -> 20.4 mm
- net /AF-2v8: track 12.9 -> 3.25 mm
- net /MCU/spi1_miso: track 19.6 -> 12.9 mm
- net /Power/2v8: track 30.4 -> 24.2 mm
- net /MCU/usart2_tx: track 4.38 -> 9.96 mm
- net Net-(JP11-B): track 8.22 -> 13.6 mm
- net /2v8: track 27.0 -> 22.0 mm
- net /Camera/DVP_VSYNC: track 41.6 -> 37.1 mm
- net /GNDA: track 11.0 -> 15.4 mm
- net /LCD/lcd_led: track 5.81 -> 10.0 mm
- net Net-(D5-K): track 0.00 -> 3.53 mm
- net Net-(D5-A): track 3.53 -> 0.00 mm
- net /DVDD-1v5: track 16.5 -> 13.1 mm
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Other:
- board size 66.4 x 47.2 mm -> 65.7 x 45.8 mm
- board text added: "1"
- board text added: "1v5"
- board text added: "24"
- board text added: "2v8"
- board text added: "3v3"
- board text added: "8"
- board text added: "A2v8"
- board text added: "AF-2v8"
- board text added: "DSI"
- board text added: "GND"
- board text added: "GrinReflex DK1"
- board text added: "REV 0.2 15.08.2025"
- board text added: "USB"
- board text added: "smps"
- board text removed: "rx"
- board text removed: "tx"
