File: v0.1/v0.1.kicad_sch (KiCad schematic)
At the start: 8 parts

Commit message: [HW] [PCB] phase #2
Parts:
- added JP10, JP11: SolderJumper_2_Open, Jumper:SolderJumper-2_P1.3mm_Open_TrianglePad1.0x1.5mm, symbol Jumper:SolderJumper_2_Open
- added R16, R17: 4.7k, Resistor_SMD:R_0603_1608Metric, symbol Device:R_Small
- added R18: 10k, Resistor_SMD:R_0603_1608Metric, symbol Device:R_Small
- added TP13: TestPoint, TestPoint:TestPoint_Pad_D1.0mm, symbol Connector:TestPoint
Connections:
- net DVDD_3V3: now also R16.1, R17.1
- net Power/3v3_pwr: now also JP10.2 (B)
- net Power/GNDA: now also JP11.2 (B)
- net AVDD-2v8: now reaches JP3.1 (A)
- net DVDD-1v5: now reaches JP2.1 (A)
- net AF-2v8: now reaches JP4.1 (A)
- net +5V: now reaches JP6.1 (A)
- net 2v8: now reaches JP1.1 (A)
- new net 3v3_pwr: JP10.1 (A)
- new net Camera/DVP_PWDN: R18.1
- new net Camera/OV_STROBE: TP13.1
- new net GND: R18.2
- new net GNDA: JP11.1 (A)
- new net I2C1_SCL: R16.2
- new net I2C1_SDA: R17.2
Other:
- added sheet Camera (camera.kicad_sch)
- sheet MCU ports: added DCMI_D[0..7], DCMI_HS, DCMI_PCLK, DCMI_VS, MCO, NRST, OSC_32IN, OSC_32OUT, OSC_IN, OSC_OUT, SWCLK, SWDIO, i2c1_scl, i2c1_sda, spi1_miso, spi1_mosi, spi1_nss, spi1_sck, usart1_rx, usart1_tx, usart2_rx, usart2_tx; removed none
- note added: "pull up i2c ?"
- moved on the sheet: JP1, JP2, JP3, JP4, JP5, JP6

Commit message: [HW] [PCB] v.01 phase #3
Parts:
- added J1: Conn_01x05_Pin, Connector_PinHeader_2.54mm:PinHeader_1x05_P2.54mm_Vertical, symbol Connector:Conn_01x05_Pin
- added J2: Conn_01x04_Pin, Connector_PinHeader_2.54mm:PinHeader_1x04_P2.54mm_Vertical, symbol Connector:Conn_01x04_Pin
- added J3, J4: Conn_01x02_Pin, Connector_PinHeader_2.54mm:PinHeader_1x02_P2.54mm_Vertical, symbol Connector:Conn_01x02_Pin
- added R3, R4: 4.7k, Resistor_SMD:R_0603_1608Metric, symbol Device:R_Small
- renumbered JP6 to JP1, JP11 to JP2, JP5 to JP3, JP3 to JP5, JP2 to JP6, JP1 to JP7, JP10 to JP8, R16 to R1, R17 to R2, R18 to R5, R1 to R6, R2 to R7, TP13 to TP1
Connections:
- net 3v3_pwr: now also R1.1, R2.1, J1.4 (Pin_4), R3.1, R4.1
- net DVDD_3V3: no longer R1.1, R2.1
- net GND: now also J1.5 (Pin_5)
- net MCU/SWCLK: now also J1.2 (Pin_2)
- net MCU/SWDIO: now also J1.3 (Pin_3)
- net MCU/spi1_miso: now also J2.4 (Pin_4)
- net MCU/spi1_mosi: now also J2.3 (Pin_3)
- net MCU/spi1_nss: now also J2.2 (Pin_2)
- net MCU/spi1_sck: now also J2.1 (Pin_1)
- net MCU/usart1_rx: now also J3.2 (Pin_2)
- net MCU/usart1_tx: now also J3.1 (Pin_1)
- net MCU/usart2_rx: now also J4.2 (Pin_2)
- net MCU/usart2_tx: now also J4.1 (Pin_1)
- net RESET: now also J1.1 (Pin_1)
- new net i2c6_scl: R4.2
- new net i2c6_sda: R3.2
Other:
- added sheet Clock_Reset (sheets/clock_reset.kicad_sch)
- sheet Camera: file camera.kicad_sch -> sheets/camera.kicad_sch
- sheet FLASH: file flash.kicad_sch -> sheets/flash.kicad_sch
- sheet LCD: file LCD.kicad_sch -> sheets/LCD.kicad_sch
- sheet MCU: file MCU.kicad_sch -> sheets/MCU.kicad_sch
- sheet MCU ports: added PB13, PB14, PB15, VDD, i2c6_scl, i2c6_sda; removed none
- sheet Power: file Power.kicad_sch -> sheets/Power.kicad_sch
- sheet USB-C: file USB.kicad_sch -> sheets/USB.kicad_sch
- moved on the sheet: R5, R6, R7, TP1

Commit message: [HW] [PCB] v0.1_Y48 revision
Parts:
- J1, J2, J3, J4, TP1: now left out of the parts list
Changed lines of the file:
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@@
 		(unit 1)
 		(exclude_from_sim no)
-		(in_bom yes)
+		(in_bom no)
 		(on_board yes)
 		(dnp no)
@@
 		(unit 1)
 		(exclude_from_sim no)
-		(in_bom yes)
+		(in_bom no)
 		(on_board yes)
 		(dnp no)
@@
 		(unit 1)
 		(exclude_from_sim no)
-		(in_bom yes)
+		(in_bom no)
 		(on_board yes)
 		(dnp no)
@@
 		(unit 1)
 		(exclude_from_sim no)
-		(in_bom yes)
+		(in_bom no)
 		(on_board yes)
 		(dnp no)
@@
 		(unit 1)
 		(exclude_from_sim no)
-		(in_bom yes)
-		(on_board yes)
-		(dnp no)
+		(in_bom no)
+		(on_board yes)
+		(dnp no)

Commit message: [HW] [PCB] revision v0.1_Y49
Parts:
- removed R3, R4: 4.7k, Resistor_SMD:R_0603_1608Metric, symbol Device:R_Small
- renumbered R5 to R3, R6 to R4, R7 to R5
Other:
- sheet Clock_Reset ports: added VCC; removed none
- sheet MCU ports: added SPI2_MOSI, SPI2_SCK; removed i2c6_scl, i2c6_sda
- sheet USB-C ports: added none; removed USBC_DETECT, USBC_FLT

Commit message: [HW] [PCB] PCB Revision 0.2_Y50; DK1
Parts:
- removed J2: Conn_01x04_Pin, Connector_PinHeader_2.54mm:PinHeader_1x04_P2.54mm_Vertical, symbol Connector:Conn_01x04_Pin
- removed JP3: SolderJumper_2_Open, Jumper:SolderJumper-2_P1.3mm_Open_TrianglePad1.0x1.5mm, symbol Jumper:SolderJumper_2_Open
- added J2, J3: Conn_01x02_Pin, Connector_PinHeader_2.54mm:PinHeader_1x02_P2.54mm_Vertical, symbol Connector:Conn_01x02_Pin
- R1, R2: footprint Resistor_SMD:R_0603_1608Metric -> Resistor_SMD:R_0402_1005Metric
- R4, R5: value 27R -> 33R
- renumbered J3 to J4, J4 to J5, JP4 to JP3, JP5 to JP4, JP6 to JP5, JP7 to JP6, JP8 to JP7
Connections:
- net MCU/spi1_miso: now also J2.2 (Pin_2)
- net MCU/spi1_mosi: now also J2.1 (Pin_1)
- net MCU/spi1_nss: now also J3.2 (Pin_2)
- net MCU/spi1_sck: now also J3.1 (Pin_1)
Other:
- sheet LCD ports: added none; removed gnd
