File: v0.1/sheets/LCD.kicad_sch (KiCad schematic)
At the start: 6 parts

Commit message: [HW] [PCB] v0.1_Y48 revision
Parts:
- Q1: LCSC Part # (none) -> C10487
- U6: LCSC Part # (none) -> C6364658
Changed lines of the file:
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@@
+			)
+		)
+		(property "LCSC Part #" "C10487"
+			(at 149.86 92.71 0)
+			(effects
+				(font
+					(size 1.27 1.27)
+				)
+				(hide yes)
 			)
 		)
@@
 			(at 189.23 93.98 0)
 			(effects
+				(font
+					(size 1.27 1.27)
+				)
+				(hide yes)
+			)
+		)
+		(property "LCSC Part #" "C6364658"
+			(at 189.23 93.98 0)
+			(effects

Commit message: [HW] [PCB] revision v0.1_Y49
Parts:
- renumbered R12 to R10, R13 to R11, R14 to R12
Changed lines of the file:
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@@
 		(dnp no)
 		(fields_autoplaced yes)
-		(property "Reference" "R12"
+		(property "Reference" "R10"
 			(at 151.13 104.1399 0)
 			(effects
@@
 			(project "v0.1"
 				(path "/d5a88f92-aedf-4ebc-b36f-cbb4d57161cd/5c0eb129-997c-46e4-80fd-8da3e9e620de"
-					(reference "R12")
+					(reference "R10")
 					(unit 1)
 				)
@@
 		(dnp no)
 		(fields_autoplaced yes)
-		(property "Reference" "R13"
+		(property "Reference" "R11"
 			(at 160.02 82.5499 0)
 			(effects
@@
 			(project ""
 				(path "/d5a88f92-aedf-4ebc-b36f-cbb4d57161cd/5c0eb129-997c-46e4-80fd-8da3e9e620de"
-					(reference "R13")
+					(reference "R11")
 					(unit 1)
 				)
@@
 		(dnp no)
 		(fields_autoplaced yes)
-		(property "Reference" "R14"
+		(property "Reference" "R12"
 			(at 182.88 120.6499 0)
 			(effects
@@
 			(project "v0.1"
 				(path "/d5a88f92-aedf-4ebc-b36f-cbb4d57161cd/5c0eb129-997c-46e4-80fd-8da3e9e620de"
-					(reference "R14")
+					(reference "R12")
 					(unit 1)
 				)

Commit message: [HW] [PCB] PCB Revision 0.2_Y50; DK1
Parts:
- R10: renamed from R12; footprint Resistor_SMD:R_0603_1608Metric -> Resistor_SMD:R_0402_1005Metric
- R11: renamed from R10; footprint Resistor_SMD:R_0603_1608Metric -> Resistor_SMD:R_0402_1005Metric
- R12: renamed from R11; footprint Resistor_SMD:R_0603_1608Metric -> Resistor_SMD:R_0402_1005Metric
- U6: footprint Grinreflex:FPC-SMD_8P-P0.50_AFC24-S08FCA-00 -> Grinreflex:FPC-SMD_8P-P0.50_FH34D-8S-0.5SH-50; LCSC Part # C6364658 -> C3169423
Other:
- moved on the sheet: C17, R10
Changed lines of the file:
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@@
+	)
+	(junction
+		(at 124.46 105.41)
+		(diameter 0)
+		(color 0 0 0 0)
 	)
 	(junction
@@
 		(color 0 0 0 0)
 	)
-	(junction
-		(at 148.59 134.62)
-		(diameter 0)
-		(color 0 0 0 0)
-	)
-	(junction
-		(at 165.1 134.62)
-		(diameter 0)
-		(color 0 0 0 0)
-	)
 	(wire
 		(pts
@@
 	(wire
 		(pts
-			(xy 172.72 87.63) (xy 185.42 87.63)
-		)
-		(stroke
-			(width 0)
-			(type default)
-		)
-	)
-	(wire
-		(pts
-			(xy 165.1 134.62) (xy 148.59 134.62)
-		)
-		(stroke
-			(width 0)
-			(type default)
-		)
-	)
-	(wire
-		(pts
 			(xy 153.67 92.71) (xy 157.48 92.71)
 		)
@@
 	(wire
 		(pts
-			(xy 180.34 125.73) (xy 180.34 134.62)
-		)
-		(stroke
-			(width 0)
-			(type default)
-		)
-	)
-	(wire
-		(pts
-			(xy 148.59 134.62) (xy 148.59 137.16)
-		)
-		(stroke
-			(width 0)
-			(type default)
-		)
-	)
-	(wire
-		(pts
-			(xy 180.34 107.95) (xy 180.34 118.11)
+			(xy 132.08 96.52) (xy 132.08 105.41)
+		)
+		(stroke
+			(width 0)
+			(type default)
+		)
+	)
+	(wire
+		(pts
+			(xy 124.46 105.41) (xy 124.46 107.95)
+		)
+		(stroke
+			(width 0)
+			(type default)
+		)
+	)
+	(wire
+		(pts
+			(xy 132.08 78.74) (xy 132.08 88.9)
 		)
 		(stroke
@@
 	(wire
 		(pts
-			(xy 165.1 125.73) (xy 165.1 134.62)
+			(xy 116.84 96.52) (xy 116.84 105.41)
 		)
 		(stroke
@@
 	(wire
 		(pts
-			(xy 165.1 113.03) (xy 165.1 118.11)
+			(xy 116.84 83.82) (xy 116.84 88.9)
 		)
 		(stroke
@@
 	(wire
 		(pts
+			(xy 168.91 87.63) (xy 185.42 87.63)
+		)
+		(stroke
+			(width 0)
+			(type default)
+		)
+	)
+	(wire
+		(pts
 			(xy 172.72 85.09) (xy 185.42 85.09)
 		)
@@
 	(wire
 		(pts
-			(xy 148.59 125.73) (xy 148.59 134.62)
-		)
-		(stroke
-			(width 0)
-			(type default)
-		)
-	)
-	(wire
-		(pts
-			(xy 180.34 134.62) (xy 165.1 134.62)
+			(xy 124.46 105.41) (xy 116.84 105.41)
+		)
+		(stroke
+			(width 0)
+			(type default)
+		)
+	)
+	(wire
+		(pts
+			(xy 132.08 105.41) (xy 124.46 105.41)
 		)
 		(stroke
@@
 		)
 	)
-	(label "LCD_GND"
-		(at 148.59 125.73 270)
-		(effects
-			(font
-				(size 1.27 1.27)
-			)
-			(justify right bottom)
-		)
-	)
-	(label "LCD_GND"
-		(at 172.72 87.63 0)
-		(effects
-			(font
-				(size 1.27 1.27)
-			)
-			(justify left bottom)
-		)
-	)
 	(label "LCD_RESET"
 		(at 172.72 90.17 0)
@@
 	)
 	(label "LCD_CS"
-		(at 180.34 115.57 90)
+		(at 132.08 86.36 90)
 		(effects
 			(font
@@
 		)
 	)
-	(hierarchical_label "gnd"
-		(shape input)
-		(at 160.02 134.62 270)
-		(effects
-			(font
-				(size 1.27 1.27)
-			)
-			(justify right)
-		)
-	)
 	(hierarchical_label "lcd_reset"
 		(shape input)
@@
 	(hierarchical_label "3v3"
 		(shape input)
-		(at 165.1 113.03 90)
+		(at 116.84 83.82 90)
 		(effects
 			(font
@@
 			)
 			(justify left)
+		)
+	)
+	(symbol
+		(lib_id "power:GND")
+		(at 168.91 87.63 270)
+		(unit 1)
+		(exclude_from_sim no)
+		(in_bom yes)
+		(on_board yes)
+		(dnp no)
+		(fields_autoplaced yes)
+		(property "Reference" "#PWR041"
+			(at 162.56 87.63 0)
+			(effects
+				(font
+					(size 1.27 1.27)
+				)
+				(hide yes)
+			)
+		)
+		(property "Value" "GND"
+			(at 165.1 87.6299 90)
+			(effects
+				(font
+					(size 1.27 1.27)
+				)
+				(justify right)
+			)
+		)
+		(property "Footprint" ""
+			(at 168.91 87.63 0)
+			(effects
+				(font
+					(size 1.27 1.27)
+				)
+				(hide yes)
+			)
+		)
+		(property "Datasheet" ""
+			(at 168.91 87.63 0)
+			(effects
+				(font
+					(size 1.27 1.27)
+				)
+				(hide yes)
+			)
+		)
+		(property "Description" "Power symbol creates a global label with name \"GND\" , ground"
+			(at 168.91 87.63 0)
+			(effects
+				(font
+					(size 1.27 1.27)
+				)
+				(hide yes)
+			)
+		)
+		(pin "1"
+		)
+		(instances
+			(project "v0.1"
+				(path "/d5a88f92-aedf-4ebc-b36f-cbb4d57161cd/5c0eb129-997c-46e4-80fd-8da3e9e620de"
+					(reference "#PWR041")
+					(unit 1)
+				)
+			)
 		)
 	)
@@
 		(dnp no)
 		(fields_autoplaced yes)
-		(property "Reference" "R10"
+		(property "Reference" "R11"
 			(at 151.13 104.1399 0)
 			(effects
@@
 			)
 		)
-		(property "Footprint" "Resistor_SMD:R_0603_1608Metric"
+		(property "Footprint" "Resistor_SMD:R_0402_1005Metric"
 			(at 146.812 105.41 90)
 			(effects
@@
 			(project "v0.1"
 				(path "/d5a88f92-aedf-4ebc-b36f-cbb4d57161cd/5c0eb129-997c-46e4-80fd-8da3e9e620de"
-					(reference "R10")
+					(reference "R11")
 					(unit 1)
 				)
@@
 	(symbol
 		(lib_id "Device:C")
-		(at 165.1 121.92 0)
+		(at 116.84 92.71 0)
 		(unit 1)
 		(exclude_from_sim no)
@@
 		(fields_autoplaced yes)
 		(property "Reference" "C17"
-			(at 168.91 120.6499 0)
+			(at 120.65 91.4399 0)
 			(effects
 				(font
@@
 		)
 		(property "Value" "10uF"
-			(at 168.91 123.1899 0)
+			(at 120.65 93.9799 0)
 			(effects
 				(font
@@
 		)
 		(property "Footprint" "Capacitor_SMD:C_0805_2012Metric"
-			(at 166.0652 125.73 0)
+			(at 117.8052 96.52 0)
 			(effects
 				(font
@@
 		)
 		(property "Datasheet" "~"
-			(at 165.1 121.92 0)
+			(at 116.84 92.71 0)
 			(effects
 				(font
@@
 		)
 		(property "Description" "Unpolarized capacitor"
-			(at 165.1 121.92 0)
+			(at 116.84 92.71 0)
 			(effects
 				(font
@@
 			)
 		)
-		(property "Footprint" "Grinreflex:FPC-SMD_8P-P0.50_AFC24-S08FCA-00"
+		(property "Footprint" "Grinreflex:FPC-SMD_8P-P0.50_FH34D-8S-0.5SH-50"
 			(at 189.23 93.98 0)
 			(effects
@@
 			)
 		)
-		(property "LCSC Part #" "C6364658"
+		(property "LCSC Part #" "C3169423"
 			(at 189.23 93.98 0)
 			(effects
@@
 		(dnp no)
 		(fields_autoplaced yes)
-		(property "Reference" "R11"
+		(property "Reference" "R12"
 			(at 160.02 82.5499 0)
 			(effects
@@
 			)
 		)
-		(property "Footprint" "Resistor_SMD:R_0603_1608Metric"
+		(property "Footprint" "Resistor_SMD:R_0402_1005Metric"
 			(at 155.702 83.82 90)
 			(effects
@@
 			(project ""
 				(path "/d5a88f92-aedf-4ebc-b36f-cbb4d57161cd/5c0eb129-997c-46e4-80fd-8da3e9e620de"
-					(reference "R11")
+					(reference "R12")
 					(unit 1)
 				)
@@
 	(symbol
 		(lib_id "Device:R")
-		(at 180.34 121.92 0)
+		(at 132.08 92.71 0)
 		(unit 1)
 		(exclude_from_sim no)
@@
 		(dnp no)
 		(fields_autoplaced yes)
-		(property "Reference" "R12"
-			(at 182.88 120.6499 0)
+		(property "Reference" "R10"
+			(at 134.62 91.4399 0)
 			(effects
 				(font
@@
 		)
 		(property "Value" "100k"
-			(at 182.88 123.1899 0)
+			(at 134.62 93.9799 0)
 			(effects
 				(font
@@
 			)
 		)
-		(property "Footprint" "Resistor_SMD:R_0603_1608Metric"
-			(at 178.562 121.92 90)
+		(property "Footprint" "Resistor_SMD:R_0402_1005Metric"
+			(at 130.302 92.71 90)
 			(effects
 				(font
@@
 		)
 		(property "Datasheet" "~"
-			(at 180.34 121.92 0)
+			(at 132.08 92.71 0)
 			(effects
 				(font
@@
 		)
 		(property "Description" "Resistor"
-			(at 180.34 121.92 0)
+			(at 132.08 92.71 0)
 			(effects
 				(font
@@
 			(project "v0.1"
 				(path "/d5a88f92-aedf-4ebc-b36f-cbb4d57161cd/5c0eb129-997c-46e4-80fd-8da3e9e620de"
-					(reference "R12")
+					(reference "R10")
 					(unit 1)
 				)
@@
 	(symbol
 		(lib_id "power:GND")
-		(at 148.59 137.16 0)
+		(at 124.46 107.95 0)
 		(unit 1)
 		(exclude_from_sim no)
@@
 		(fields_autoplaced yes)
 		(property "Reference" "#PWR029"
-			(at 148.59 143.51 0)
+			(at 124.46 114.3 0)
 			(effects
 				(font
@@
 		)
 		(property "Value" "GND"
-			(at 148.59 142.24 0)
+			(at 124.46 113.03 0)
 			(effects
 				(font
@@
 		)
 		(property "Footprint" ""
-			(at 148.59 137.16 0)
+			(at 124.46 107.95 0)
 			(effects
 				(font
@@
 		)
 		(property "Datasheet" ""
-			(at 148.59 137.16 0)
+			(at 124.46 107.95 0)
 			(effects
 				(font
@@
 		)
 		(property "Description" "Power symbol creates a global label with name \"GND\" , ground"
-			(at 148.59 137.16 0)
-			(effects
-				(font
+			(at 124.46 107.95 0)
+			(effects
+				(font
