File: v0.1/sheets/MCU.kicad_sch (KiCad schematic)
At the start: 28 parts, among them U10 STM32U5G9ZJTxQ

Commit message: [HW] [PCB] v.01 phase #3
Parts:
- removed C27: 10uf, Capacitor_SMD:C_0805_2012Metric, symbol Device:C_Small
- removed C28, C29, C30, C31, C32, C33, C34, C35, C36, C37: 100nf, Capacitor_SMD:C_0603_1608Metric, symbol Device:C_Small
- renumbered C38 to C27, C39 to C28, C40 to C29, C41 to C30, C42 to C31, C43 to C32, C44 to C33, C45 to C34, C46 to C35, C47 to C36, C48 to C37
Other:
- moved on the sheet: L7, R20

Commit message: [HW] [PCB] v0.1_Y48 revision
Parts:
- U10: LCSC Part # (none) -> C22445371
Connections:
- net NRST: now also U10.28 (NRST); no longer U10.134 (PB4)
Changed lines of the file:
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@@
 	(wire
 		(pts
-			(xy 104.14 33.02) (xy 104.14 55.88)
-		)
-		(stroke
-			(width 0)
-			(type default)
-		)
-	)
-	(wire
-		(pts
 			(xy 106.68 137.16) (xy 106.68 149.86)
 		)
@@
 		)
 	)
+	(wire
+		(pts
+			(xy 50.8 137.16) (xy 50.8 142.24)
+		)
+		(stroke
+			(width 0)
+			(type default)
+		)
+	)
 	(label "HSPI1_SIO7"
 		(at 83.82 149.86 90)
@@
 		)
 	)
+	(hierarchical_label "NRST"
+		(shape input)
+		(at 50.8 142.24 270)
+		(effects
+			(font
+				(size 1.27 1.27)
+			)
+			(justify right)
+		)
+	)
 	(hierarchical_label "PB14"
 		(shape input)
@@
 		)
 	)
-	(hierarchical_label "NRST"
-		(shape input)
-		(at 104.14 33.02 90)
-		(effects
-			(font
-				(size 1.27 1.27)
-			)
-			(justify left)
-		)
-	)
 	(symbol
 		(lib_id "Device:C_Small")
@@
 			(effects
 				(font
+					(size 1.27 1.27)
+				)
+				(hide yes)
+			)
+		)
+		(property "LCSC Part #" "C22445371"
+			(at 132.08 96.52 90)
+			(effects
+				(font

Commit message: [HW] [PCB] revision v0.1_Y49
Parts:
- added C27: 10uf, Capacitor_SMD:C_0805_2012Metric, symbol Device:C_Small
- added C28, C29, C30, C31, C32, C33, C34, C35, C36, C37, C38: 100nf, Capacitor_SMD:C_0603_1608Metric, symbol Device:C_Small
- added TP19, TP20, TP21, TP22: TestPoint, TestPoint:TestPoint_Pad_D1.0mm, symbol Connector:TestPoint
- renumbered C27 to C39, C28 to C40, C29 to C41, C30 to C42, C31 to C43, C32 to C44, C33 to C45, C34 to C46, C35 to C47, C36 to C48, C37 to C49, JP11 to JP10, JP12 to JP11, JP10 to JP9, R20 to R16
Connections:
- net GND: now also C27.2, C28.1, C29.2, C30.1, C31.2, C32.1, C33.2, C34.1, C35.2, C36.1, C37.2, C38.1
- net VDD: now also C27.1, C28.2, C29.1, C30.2, C31.1, C32.2, C33.1, C34.2, C35.1, C36.2, C37.1, C38.2
- net at U10.1 (PE2): now also TP19.1
- net SPI2_MOSI: now reaches U10.119 (PD3)
- net SPI2_SCK: now reaches U10.120 (PD4)
- net at U10.2 (PE3): now also TP20.1
- net at U10.4 (PE5): now also TP21.1
- net at U10.5 (PE6): now also TP22.1
- net DCMI_D8: no longer names the net of U10.113 (PC10)
- net i2c6_scl: no longer names the net of U10.117 (PD1)
- net i2c6_sda: no longer names the net of U10.116 (PD0)
Other:
- moved on the sheet: L7, R16

Commit message: [HW] [PCB] PCB Revision 0.2_Y50; DK1
Parts:
- C47, C49: footprint Capacitor_SMD:C_0603_1608Metric -> Capacitor_SMD:C_0402_1005Metric
- R16: footprint Resistor_SMD:R_0603_1608Metric -> Resistor_SMD:R_0402_1005Metric
- renumbered JP11 to JP10, JP9 to JP8, JP10 to JP9
Connections:
- net SPI2_MOSI: now also U10.120 (PD4); no longer U10.119 (PD3)
- net SPI2_SCK: now also U10.119 (PD3); no longer U10.120 (PD4)
Changed lines of the file:
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@@
 	(wire
 		(pts
-			(xy 180.34 31.75) (xy 180.34 55.88)
-		)
-		(stroke
-			(width 0)
-			(type default)
-		)
-	)
-	(wire
-		(pts
 			(xy 111.76 137.16) (xy 111.76 149.86)
 		)
@@
 	(wire
 		(pts
+			(xy 182.88 31.75) (xy 182.88 55.88)
+		)
+		(stroke
+			(width 0)
+			(type default)
+		)
+	)
+	(wire
+		(pts
 			(xy 111.76 38.1) (xy 111.76 55.88)
 		)
@@
 	(wire
 		(pts
-			(xy 193.04 40.64) (xy 193.04 55.88)
+			(xy 193.04 31.75) (xy 193.04 55.88)
+		)
+		(stroke
+			(width 0)
+			(type default)
+		)
+	)
+	(wire
+		(pts
+			(xy 180.34 31.75) (xy 180.34 55.88)
 		)
 		(stroke
@@
 	(wire
 		(pts
-			(xy 195.58 40.64) (xy 195.58 55.88)
+			(xy 195.58 31.75) (xy 195.58 55.88)
 		)
 		(stroke
@@
 	(wire
 		(pts
-			(xy 101.6 137.16) (xy 101.6 156.21)
+			(xy 101.6 137.16) (xy 101.6 176.53)
 		)
 		(stroke
@@
 		)
 	)
-	(wire
-		(pts
-			(xy 182.88 31.75) (xy 182.88 55.88)
-		)
-		(stroke
-			(width 0)
-			(type default)
-		)
-	)
 	(bus
 		(pts
@@
 	(hierarchical_label "DCMI_PCLK"
 		(shape input)
-		(at 195.58 40.64 90)
+		(at 195.58 31.75 90)
 		(effects
 			(font
 				(size 1.27 1.27)
+				(color 255 0 15 1)
 			)
 			(justify left)
@@
 	(hierarchical_label "hspi1_ncs"
 		(shape input)
-		(at 101.6 156.21 270)
+		(at 101.6 176.53 270)
 		(effects
 			(font
@@
 	(hierarchical_label "DCMI_HS"
 		(shape input)
-		(at 193.04 40.64 90)
+		(at 193.04 31.75 90)
 		(effects
 			(font
 				(size 1.27 1.27)
+				(color 255 0 7 1)
 			)
 			(justify left)
@@
 	(hierarchical_label "SPI2_MOSI"
 		(shape output)
-		(at 180.34 31.75 90)
+		(at 182.88 31.75 90)
 		(effects
 			(font
@@
 			(font
 				(size 1.27 1.27)
+				(color 255 0 7 1)
 			)
 			(justify left)
@@
 	(hierarchical_label "SPI2_SCK"
 		(shape output)
-		(at 182.88 31.75 90)
+		(at 180.34 31.75 90)
 		(effects
 			(font
@@
 			)
 		)
-		(property "Footprint" "Capacitor_SMD:C_0603_1608Metric"
+		(property "Footprint" "Capacitor_SMD:C_0402_1005Metric"
 			(at 271.78 27.94 0)
 			(effects
@@
 		(on_board yes)
 		(dnp no)
-		(property "Reference" "JP9"
+		(property "Reference" "JP8"
 			(at 19.304 74.676 0)
 			(effects
@@
 			(project "v0.1"
 				(path "/d5a88f92-aedf-4ebc-b36f-cbb4d57161cd/c6246201-b9a6-4df1-a90f-d6ccbe22ca4d"
-					(reference "JP9")
+					(reference "JP8")
 					(unit 1)
 				)
@@
 		(on_board yes)
 		(dnp no)
-		(property "Reference" "JP11"
+		(property "Reference" "JP10"
 			(at 24.638 69.85 0)
 			(effects
@@
 			(project "v0.1"
 				(path "/d5a88f92-aedf-4ebc-b36f-cbb4d57161cd/c6246201-b9a6-4df1-a90f-d6ccbe22ca4d"
-					(reference "JP11")
+					(reference "JP10")
 					(unit 1)
 				)
@@
 		(on_board yes)
 		(dnp no)
-		(property "Reference" "JP10"
+		(property "Reference" "JP9"
 			(at 26.416 77.724 0)
 			(effects
@@
 			(project "v0.1"
 				(path "/d5a88f92-aedf-4ebc-b36f-cbb4d57161cd/c6246201-b9a6-4df1-a90f-d6ccbe22ca4d"
-					(reference "JP10")
+					(reference "JP9")
 					(unit 1)
 				)
@@
 			)
 		)
-		(property "Footprint" "Resistor_SMD:R_0603_1608Metric"
+		(property "Footprint" "Resistor_SMD:R_0402_1005Metric"
 			(at 99.06 162.56 0)
 			(effects
@@
 			)
 		)
-		(property "Footprint" "Capacitor_SMD:C_0603_1608Metric"
+		(property "Footprint" "Capacitor_SMD:C_0402_1005Metric"
 			(at 262.89 27.94 0)
 			(effects
