File: v0.1/sheets/Power.kicad_sch (KiCad schematic)
At the start: 38 parts, among them U1 XC6206P152MR, U2 XC6206P282MR, U3 SY8088AAC, U4 XC6206P282MR

Commit message: [HW] [PCB] v.01 phase #3
Parts:
- renumbered 2v8-TP1 to TP2, AF-2v8-TP1 to TP3, 1v5-TP1 to TP4, 3v3-TP1 to TP5, GNDA-1TP1 to TP6
Other:
- moved on the sheet: C15, C16, R11, U5

Commit message: [HW] [PCB] v0.1_Y48 revision
Parts:
- D1: LCSC Part # (none) -> C383210
- D3: footprint Diode_SMD:D_SOD-323 -> Grinreflex:SOD-523F_L1.2-W0.8-LS1.7-RD; LCSC Part # (none) -> C136161
- L3: LCSC Part # (none) -> C36400
- TP2, TP3, TP4, TP5, TP6: now left out of the parts list
- U1: LCSC Part # (none) -> C56110
- U2, U4: LCSC Part # (none) -> C479055
- U3: LCSC Part # (none) -> C79313
- U5: LCSC Part # (none) -> C2969933

Commit message: [HW] [PCB] revision v0.1_Y49
Parts:
- R6: renamed from R8; footprint Resistor_SMD:R_0603_1608Metric -> Resistor_SMD:R_0402_1005Metric
- R7: renamed from R9; footprint Resistor_SMD:R_0603_1608Metric -> Resistor_SMD:R_0402_1005Metric
- renumbered R10 to R8, R11 to R9
