File: v0.1/sheets/USB.kicad_sch (KiCad schematic)
At the start: 17 parts

Commit message: [HW] [PCB] v.01 phase #3
Parts:
- renumbered 5V_USB_TP1 to TP7
Changed lines of the file:
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@@
 			"AHoAAABzAAAAaQAAACsAAABKAAAAdwAAAC8AAABpAAAAVQAAAFQAAABvAAAAcwAAAEkAAABBAAAA"
 			"QQAAAEEAAABBAAAAQQAAAEEAAABBAAAAQQAAAEEAAABBAAAAOAAAAEIAAAB2AAAAVAAAADEAAAA5"
-			"AAAAUAAAAHIAAAA3AAAAdQAAAGwAAABoADIgNDAuNjQpCgkJKHNpemUgMi41NCAtMi41NCkKCQko"
-			"c3Ryb2tlCgkJCSh3aWR0aCAwKQoJCQkodHlwZSBkZWZhdWx0KQoJCSkKCQkodXVpZCAiNTc2ZDA2"
-			"YTUtZjVjNy00NGJkLTg4NWItZTZhNDM5MDEwZmU2IikKCSkKCShidXNfZW50cnkKCQkoYXQgODMu"
-			"ODIgMTQ5Ljg2KQoJCShzaXplIC0yLjU0IDIuNTQpCgkJKHN0cm9rZQoJCQkod2lkdGggMCkKCQkJ"
-			"KHR5cGUgZGVmYXVsdCkKCQkpCgkJKHV1aWQgIjc0MDY2Y2U5LTNmODUtNGQ4ZC1iZmQ0LTY3OGVm"
-			"YjE4OGI5ZSIpCgkpCgkoYnVzX2VudHJ5CgkJKGF0IDE0OS44NiA0MC42NCkKCQkoc2l6ZSAyLjU0"
-			"IC0yLjU0KQoJCShzdHJva2UKCQkJKHdpZHRoIDApCgkJCSh0eXBlIGRlZmF1bHQpCgkJKQoJCSh1"
-			"dWlkICI3ZGZjNWNhZC03MmZlLTRlOWYtODE3ZS02MjNmYTZmMGIxNDMiKQoJKQoJKGJ1c19lbnRy"
-			"eQoJCShhdCAxNTIuNCA0MC42NCkKCQkoc2l6ZSAyLjU0IC0yLjU0KQoJCShzdHJva2UKCQkJKHdp"
-			"ZHRoIDApCgkJCSh0eXBlIGRlZmF1bHQpCgkJKQoJCSh1dWlkICI3ZjE3MmY1Mi00ODhkLTQ4ZTgt"
-			"YTU3ZS00NzBkZDc2M2EzOWQiKQoJKQoJKGJ1c19lbnRyeQoJCShhdCAxNDQuNzggNDAuNjQpCgkJ"
-			"KHNpemUgMi41NCAtMi41NCkKCQkoc3Ryb2tlCgkJCSh3aWR0aCAwKQoJCQkodHlwZSBkZWZhdWx0"
-			"KQoJCSkKCQkodXVpZCAiYTEyNTk0ZjktYTAzZC00YzM0LTg0NzUtYjFlNTA4MzRiYmIzIikKCSkK"
-			"CShidXNfZW50cnkKCQkoYXQgMTA5LjIyIDE0OS44NikKCQkoc2l6ZSAyLjU0IDIuNTQpCgkJKHN0"
-			"cm9rZQoJCQkod2lkdGggMCkKCQkJKHR5cGUgZGVmYXVsdCkKCQkpCgkJKHV1aWQgImFjMmFmYjI4"
-			"LTBiMWQtNDk0MC04MzU2LWMzODFlYmQ2ZjQ1ZSIpCgkpCgkoYnVzX2VudHJ5CgkJKGF0IDgxLjI4"
-			"IDE0OS44NikKCQkoc2l6ZSAtMi41NCAyLjU0KQoJCShzdHJva2UKCQkJKHdpZHRoIDApCgkJCSh0"
-			"eXBlIGRlZmF1bHQpCgkJKQoJCSh1dWlkICJjMGE1Mjg5MS00MWMyLTQzMjUtOTU4MC0wNGNjOWQw"
-			"MGE1OTgiKQoJKQoJKGJ1c19lbnRyeQoJCQ=="
+			"AAAAUAAAAHIAAAA3AAAAdQAAAGwAAABoAAAAKwAAAEkAAABBAAAAMQAAAGIAAABnAAAAQgAAAG4A"
+			"AABOAAAAQgAAAHIAAAA1AAAAMwAAAHAAAAAwAAAAUgAAADEAAAA2AAAANwAAAEgAAABIAAAAZgAA"
+			"ADAAAABuAAAAbQAAAHMAAABQAAAAaAAAAEcAAAB4AAAAcgAAAEkAAAA5AAAAZQAAADIAAABqAAAA"
+			"YgAAADIAAABnAAAAbwAAAEYAAAB4AAAATwAAAGIAAABYAAAAMQAAAG4AAABKAAAAUgAAAGcAAABo"
+			"AAAAOQAAAC8AAAAxAAAANQAAAGsAAABZAAAAaQAAAEsAAABQAAAARQAAAEMAAABLAAAAVAAAAGkA"
+			"AABaAAAAYwAAAHUAAABEAAAASQAAAHAAAABQAAAASwAAAEUAAABZAAAASQAAAHYAAABYAAAANgAA"
+			"AFQAAAAxAAAAYQAAAE8AAAA3AAAAagAAAG0AAABBAAAARQAAAEMAAABwAAAAawAAAFkAAABHAAAA"
+			"RwAAAEMAAABPAAAANAAAAHkAAABVAAAAQQAAAEEAAABBAAAAQQAAAEEAAABBAAAAQQAAAEEAAABB"
+			"AAAAQQAAAEEAAABDAAAALwAAAEMAAAB4AAAASwAAAEoAAABKAAAAUAAAAHoAAABZAAAATgAAAGwA"
+			"AABCAAAATAAAAEEAAABwAAAAMwAAAEMAAABvAAAASQAAAEgAAABHAAAAZwAAAHcAAABZAAAAYQAA"
+			"ADEAAAAyAAAANgAAAHgAAAB0AAAARgAAAEMAAAB5AAAAdAAAAEYAAABDAAAAcQAAADAAAAAwAAAA"
+			"MQAAAFIAAABrAAAAYQAAADYAAABvAAAAUwAAAEUAAABjAAAASQAAAGoAAABSAAAAawAAAE4AAABO"
+			"AAAANgAAAGcAAABHAAAAQQAAAEEAAABBAAAAQQAAAEEAAABBAAAAQQAAAEEAAABBAAAAQQAAAEIA"
+			"AABhAAAAegAAAGMAAABlAAAANwAAAFoAAAA4AAAAagAAADUAAABNAAAANAAAAGEAAABHAAAAYgAA"
+			"AGQAAAArAAAATwAAAEgAAABkAAAAYQAAADQAAABBAAAAUQAAAEEAAABBAAAAQQAAAEEAAABBAAAA"
+			"QQAAAEEAAABBAAAAQQAAAEEAAABBAAAAUAAAAHgAAABYAAAAMAAAAEcAAABnAAAAMAAAAEUAAAB4"
+			"AAAATgAAAGoAAABRAAAAagAAAHQAAAAyAAAAaQAAAG8AAABGAAAANQAAAFMAAABRAAAAQgAAAFAA"
+			"AAA2AAAAOAAAAGcAAAAwAAAAdgAAAEMAAABPAAAASQAAAHYAAAB6AAAAWAAAAGMAAABhAAAAcgAA"
+			"AHcAAABqAAAAQQAAAEEAAABBAAAAQQAAAA=="
 		)
 	)
@@
 		(dnp no)
 		(fields_autoplaced yes)
-		(property "Reference" "#PWR036"
+		(property "Reference" "#PWR037"
 			(at 148.59 43.18 0)
 			(effects
@@
 			(project "v0.1"
 				(path "/d5a88f92-aedf-4ebc-b36f-cbb4d57161cd/da524e3a-9ae7-47c3-a964-34a843fee879"
-					(reference "#PWR036")
+					(reference "#PWR037")
 					(unit 1)
 				)
@@
 		)
 		(instances
-			(project "v0.1"
+			(project ""
 				(path "/d5a88f92-aedf-4ebc-b36f-cbb4d57161cd/da524e3a-9ae7-47c3-a964-34a843fee879"
 					(reference "Q2")
@@
 		)
 		(instances
-			(project "v0.1"
+			(project ""
 				(path "/d5a88f92-aedf-4ebc-b36f-cbb4d57161cd/da524e3a-9ae7-47c3-a964-34a843fee879"
 					(reference "D4")
@@
 		)
 		(instances
-			(project "v0.1"
+			(project ""
 				(path "/d5a88f92-aedf-4ebc-b36f-cbb4d57161cd/da524e3a-9ae7-47c3-a964-34a843fee879"
 					(reference "U8")
@@
 		(dnp no)
 		(fields_autoplaced yes)
-		(property "Reference" "#PWR033"
+		(property "Reference" "#PWR034"
 			(at 110.49 80.01 0)
 			(effects
@@
 			(project "v0.1"
 				(path "/d5a88f92-aedf-4ebc-b36f-cbb4d57161cd/da524e3a-9ae7-47c3-a964-34a843fee879"
-					(reference "#PWR033")
+					(reference "#PWR034")
 					(unit 1)
 				)
@@
 		(dnp no)
 		(fields_autoplaced yes)
-		(property "Reference" "#PWR034"
+		(property "Reference" "#PWR035"
 			(at 152.4 54.61 0)
 			(effects
@@
 			(project "v0.1"
 				(path "/d5a88f92-aedf-4ebc-b36f-cbb4d57161cd/da524e3a-9ae7-47c3-a964-34a843fee879"
-					(reference "#PWR034")
+					(reference "#PWR035")
 					(unit 1)
 				)
@@
 		(dnp no)
 		(fields_autoplaced yes)
-		(property "Reference" "#PWR041"
+		(property "Reference" "#PWR042"
 			(at 222.25 102.87 0)
 			(effects
@@
 			(project "v0.1"
 				(path "/d5a88f92-aedf-4ebc-b36f-cbb4d57161cd/da524e3a-9ae7-47c3-a964-34a843fee879"
-					(reference "#PWR041")
+					(reference "#PWR042")
 					(unit 1)
 				)
@@
 		(dnp no)
 		(fields_autoplaced yes)
-		(property "Reference" "#PWR039"
+		(property "Reference" "#PWR040"
 			(at 187.96 44.45 0)
 			(effects
@@
 			(project "v0.1"
 				(path "/d5a88f92-aedf-4ebc-b36f-cbb4d57161cd/da524e3a-9ae7-47c3-a964-34a843fee879"
-					(reference "#PWR039")
+					(reference "#PWR040")
 					(unit 1)
 				)
@@
 		(dnp no)
 		(fields_autoplaced yes)
-		(property "Reference" "#PWR040"
+		(property "Reference" "#PWR041"
 			(at 207.01 54.61 0)
 			(effects
@@
 			(project "v0.1"
 				(path "/d5a88f92-aedf-4ebc-b36f-cbb4d57161cd/da524e3a-9ae7-47c3-a964-34a843fee879"
-					(reference "#PWR040")
+					(reference "#PWR041")
 					(unit 1)
 				)
@@
 		)
 		(instances
-			(project "v0.1"
+			(project ""
 				(path "/d5a88f92-aedf-4ebc-b36f-cbb4d57161cd/da524e3a-9ae7-47c3-a964-34a843fee879"
 					(reference "D5")
@@
 		(dnp no)
 		(fields_autoplaced yes)
-		(property "Reference" "#PWR032"
+		(property "Reference" "#PWR033"
 			(at 110.49 52.07 0)
 			(effects
@@
 		)
 		(instances
-			(project "v0.1"
-				(path "/d5a88f92-aedf-4ebc-b36f-cbb4d57161cd/da524e3a-9ae7-47c3-a964-34a843fee879"
-					(reference "#PWR032")
+			(project ""
+				(path "/d5a88f92-aedf-4ebc-b36f-cbb4d57161cd/da524e3a-9ae7-47c3-a964-34a843fee879"
+					(reference "#PWR033")
 					(unit 1)
 				)
@@
 		(dnp no)
 		(fields_autoplaced yes)
-		(property "Reference" "#PWR031"
+		(property "Reference" "#PWR032"
 			(at 105.41 119.38 0)
 			(effects
@@
 			(project "v0.1"
 				(path "/d5a88f92-aedf-4ebc-b36f-cbb4d57161cd/da524e3a-9ae7-47c3-a964-34a843fee879"
-					(reference "#PWR031")
+					(reference "#PWR032")
 					(unit 1)
 				)
@@
 		(dnp no)
 		(fields_autoplaced yes)
-		(property "Reference" "5V_USB_TP1"
+		(property "Reference" "TP7"
 			(at 209.55 17.0179 0)
 			(effects
@@
 			(project "v0.1"
 				(path "/d5a88f92-aedf-4ebc-b36f-cbb4d57161cd/da524e3a-9ae7-47c3-a964-34a843fee879"
-					(reference "5V_USB_TP1")
+					(reference "TP7")
 					(unit 1)
 				)
@@
 		)
 		(instances
-			(project "v0.1"
+			(project ""
 				(path "/d5a88f92-aedf-4ebc-b36f-cbb4d57161cd/da524e3a-9ae7-47c3-a964-34a843fee879"
 					(reference "U7")
@@
 		(dnp no)
 		(fields_autoplaced yes)
-		(property "Reference" "#PWR035"
+		(property "Reference" "#PWR036"
 			(at 153.67 80.01 0)
 			(effects
@@
 			(project "v0.1"
 				(path "/d5a88f92-aedf-4ebc-b36f-cbb4d57161cd/da524e3a-9ae7-47c3-a964-34a843fee879"
-					(reference "#PWR035")
+					(reference "#PWR036")
 					(unit 1)
 				)
@@
 		(dnp no)
 		(fields_autoplaced yes)
-		(property "Reference" "#PWR043"
+		(property "Reference" "#PWR044"
 			(at 236.22 92.71 0)
 			(effects
@@
 			(project "v0.1"
 				(path "/d5a88f92-aedf-4ebc-b36f-cbb4d57161cd/da524e3a-9ae7-47c3-a964-34a843fee879"
-					(reference "#PWR043")
+					(reference "#PWR044")
 					(unit 1)
 				)
@@
 		)
 		(instances
-			(project "v0.1"
+			(project ""
 				(path "/d5a88f92-aedf-4ebc-b36f-cbb4d57161cd/da524e3a-9ae7-47c3-a964-34a843fee879"
 					(reference "L6")
@@
 		(on_board yes)
 		(dnp no)
-		(property "Reference" "#PWR038"
+		(property "Reference" "#PWR039"
 			(at 179.07 63.5 0)
 			(effects
@@
 			(project "v0.1"
 				(path "/d5a88f92-aedf-4ebc-b36f-cbb4d57161cd/da524e3a-9ae7-47c3-a964-34a843fee879"
-					(reference "#PWR038")
+					(reference "#PWR039")
 					(unit 1)
 				)
@@
 		(dnp no)
 		(fields_autoplaced yes)
-		(property "Reference" "#PWR037"
+		(property "Reference" "#PWR038"
 			(at 170.18 93.98 0)
 			(effects
@@
 			(project "v0.1"
 				(path "/d5a88f92-aedf-4ebc-b36f-cbb4d57161cd/da524e3a-9ae7-47c3-a964-34a843fee879"
-					(reference "#PWR037")
+					(reference "#PWR038")
 					(unit 1)
 				)
@@
 		(dnp no)
 		(fields_autoplaced yes)
-		(property "Reference" "#PWR042"
+		(property "Reference" "#PWR043"
 			(at 234.95 58.42 0)
 			(effects
@@
 			(project "v0.1"
 				(path "/d5a88f92-aedf-4ebc-b36f-cbb4d57161cd/da524e3a-9ae7-47c3-a964-34a843fee879"
-					(reference "#PWR042")
-					(unit 1)
-				)
+					(reference "#PWR043")
+					(unit 1)
+				)

Commit message: [HW] [PCB] v0.1_Y48 revision
Parts:
- D4: LCSC Part # (none) -> C1974707
- L6: LCSC Part # (none) -> C2651144
- Q2: LCSC Part # (none) -> C2965326
- TP7: now left out of the parts list
- U7: LCSC Part # (none) -> C2927037
- U8: LCSC Part # (none) -> C1121848
Changed lines of the file:
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@@
+			)
+		)
+		(property "LCSC Part #" "C2965326"
+			(at 173.99 29.21 90)
+			(effects
+				(font
+					(size 1.27 1.27)
+				)
+				(hide yes)
 			)
 		)
@@
 			)
 		)
+		(property "LCSC Part #" "C1974707"
+			(at 114.3 105.41 90)
+			(effects
+				(font
+					(size 1.27 1.27)
+				)
+				(hide yes)
+			)
+		)
 		(pin "2"
 		)
@@
 			)
 		)
+		(property "LCSC Part #" "C1121848"
+			(at 204.47 66.04 0)
+			(effects
+				(font
+					(size 1.27 1.27)
+				)
+				(hide yes)
+			)
+		)
 		(pin "3"
 		)
@@
 		(unit 1)
 		(exclude_from_sim no)
-		(in_bom yes)
+		(in_bom no)
 		(on_board yes)
 		(dnp no)
@@
 			)
 		)
+		(property "LCSC Part #" "C2927037"
+			(at 128.27 64.77 0)
+			(effects
+				(font
+					(size 1.27 1.27)
+				)
+				(hide yes)
+			)
+		)
 		(pin "4"
 		)
@@
 			(at 199.39 105.41 0)
 			(effects
+				(font
+					(size 1.27 1.27)
+				)
+				(hide yes)
+			)
+		)
+		(property "LCSC Part #" "C2651144"
+			(at 199.39 105.41 0)
+			(effects

Commit message: [HW] [PCB] revision v0.1_Y49
Parts:
- removed JP9: SolderJumper_2_Open, Jumper:SolderJumper-2_P1.3mm_Open_TrianglePad1.0x1.5mm, symbol Jumper:SolderJumper_2_Open
- removed R17: 110k, Resistor_SMD:R_0603_1608Metric, symbol Device:R_Small
- removed R18: 200k, Resistor_SMD:R_0603_1608Metric, symbol Device:R_Small
- R13: renamed from R15; footprint Resistor_SMD:R_0603_1608Metric -> Resistor_SMD:R_0402_1005Metric
- R14: renamed from R16; footprint Resistor_SMD:R_0603_1608Metric -> Resistor_SMD:R_0402_1005Metric
Other:
- moved on the sheet: C18, C19, C20, C21, C22, D4, D5, L6, Q2, R13, R14, TP7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

Commit message: [HW] [PCB] PCB Revision 0.2_Y50; DK1
Connections:
- net VBUS: now also D5.2 (A); no longer D5.1 (K)
- net at C22.1, U8.8 (IN_GD): now also D5.1 (K); no longer D5.2 (A)
Other:
- moved on the sheet: D5
Changed lines of the file:
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@@
 	)
 	(junction
-		(at 114.3 53.34)
+		(at 163.83 60.96)
 		(diameter 0)
 		(color 0 0 0 0)
 	)
 	(junction
-		(at 163.83 60.96)
+		(at 114.3 53.34)
 		(diameter 0)
 		(color 0 0 0 0)
@@
 	(wire
 		(pts
-			(xy 19.05 31.75) (xy 31.75 31.75)
+			(xy 163.83 60.96) (xy 166.37 60.96)
 		)
 		(stroke
@@
 	(wire
 		(pts
-			(xy 153.67 48.26) (xy 156.21 48.26)
+			(xy 19.05 31.75) (xy 31.75 31.75)
 		)
 		(stroke
@@
 	(wire
 		(pts
-			(xy 116.84 27.94) (xy 116.84 30.48)
+			(xy 153.67 48.26) (xy 156.21 48.26)
 		)
 		(stroke
@@
 	(wire
 		(pts
-			(xy 153.67 55.88) (xy 153.67 50.8)
+			(xy 116.84 27.94) (xy 116.84 30.48)
 		)
 		(stroke
@@
 	(wire
 		(pts
-			(xy 163.83 60.96) (xy 165.1 60.96)
+			(xy 153.67 55.88) (xy 153.67 50.8)
 		)
 		(stroke
@@
 	(wire
 		(pts
-			(xy 172.72 60.96) (xy 177.8 60.96)
-		)
-		(stroke
-			(width 0)
-			(type default)
-		)
-	)
-	(wire
-		(pts
 			(xy 116.84 58.42) (xy 109.22 58.42)
 		)
@@
 	(wire
 		(pts
+			(xy 173.99 60.96) (xy 180.34 60.96)
+		)
+		(stroke
+			(width 0)
+			(type default)
+		)
+	)
+	(wire
+		(pts
 			(xy 101.6 40.64) (xy 102.87 40.64)
 		)
@@
 			"AAAATgAAAGoAAABRAAAAagAAAHQAAAAyAAAAaQAAAG8AAABGAAAANQAAAFMAAABRAAAAQgAAAFAA"
 			"AAA2AAAAOAAAAGcAAAAwAAAAdgAAAEMAAABPAAAASQAAAHYAAAB6AAAAWAAAAGMAAABhAAAAcgAA"
-			"AHcAAABqAAAAQQAAAEEAAABBAAAAQQAAAA=="
+			"AHcAAABqAAAAQQAAAEEAAABBAAAAQQAAAGwAAABTAAAAMAAAAHQAAABtAAAANAAAADMAAABSAAAA"
+			"NAAAAEMAAABrAAAAWQAAAHkAAABrAAAAbwAAAEkAAABvAAAAYwAAAEsAAAA0AAAAKwAAAE0AAAA4"
+			"AAAAaAAAAEYAAAAyAAAAcAAAAEsAAABTAAAAMgAAAG0AAAB5AAAAcwAAAHIAAABJAAAANgAAAE8A"
+			"AABtAAAAVwAAAFoAAABtAAAAZQAAADcAAABMAAAAbAAAAHcAAABwAAAAZQAAAGwAAABSAAAAVAAA"
+			"ADIAAABtAAAARgAAAGQAAABUAAAAWQAAADkAAABUAAAAYwAAAEoAAAB6AAAAUAAAADUAAAB5AAAA"
+			"ZAAAAE8AAABFAAAAZQAAAC8AAABjAAAASgAAAEoAAABKAAAASwAAAEUAAABsAAAASgAAAFMAAABj"
+			"AAAAdgAAAGgAAAA2AAAANwAAAG8AAAB0AAAASgAAAHUAAAAwAAAAbwAAAFQAAAAyAAAAZgAAAHUA"
+			"AABKAAAAKwAAAEUAAAAzAAAAZgAAAHYAAAAzAAAAWAAAAC8AAAAxAAAAKwAAAG8AAAAzAAAAdwAA"
+			"AGEAAABiAAAAKwAAACsAAABmAAAAYgAAAHEAAAA2AAAATwAAAE8AAABPAAAAWQAAAEIAAAAzAAAA"
+			"UwAAAFEAAABsAAAANgAAADkAAABlAAAALwAAADMAAABNAAAAOAAAAFMAAABFAAAATgAAAEQAAABZ"
+			"AAAAOAAAAEsAAAA0AAAAcwAAAFEAAABZAAAARwAAACsAAABuAAAAagAAAEgAAABBAAAAUQAAAEEA"
+			"AABBAAAAQQAAAE0AAABSAAAAUQAAAFYAAABQAAAAVAAAAEgAAAB1AAAAZgAAAE0AAABYAAAAMgAA"
+			"AHQAAAByAAAAYQAAAHUAAABIAAAAZAAAAHoAAAB3AAAAegAAAHMAAABMAAAARQAAAEIAAABNAAAA"
+			"dwAAAEwAAAB3AAAAbQAAADAAAABCAAAAWQAAAC8AAABIAAAAVwAAADcAAABiAAAAaQAAAHoAAAA3"
+			"AAAAUAAAAG4AAABnAAAAdQAAAHMAAABmAAAAeQAAAHMAAAA3AAAATwAAACsAAABXAAAAUAAAADIA"
+			"AAAzAAAASgAAAFMAAABVAAAAMQAAAEYAAAArAAAAZgAAAEMAAAByAAAAVAAAAGYAAAByAAAAdAAA"
+			"ADEAAAA3AAAAZAAAACsAAAB6AAAAYwAAAFUAAAA2AAAAZgAAAHgAAAAxAAAATwAAAG0AAAB6AAAA"
+			"RgAAAFIAAABVAAAAVgAAAFgAAABDAAAANgAAAFgAAABRAAAAQwAAAEIAAAAwAAAAYwAAADMAAABQ"
+			"AAAARgAAAEoAAABWAAAAaQAAAEQAAABGAA=="
 		)
 	)
@@
 	)
 	(label "VBUS"
-		(at 177.8 60.96 180)
+		(at 180.34 60.96 180)
 		(effects
 			(font
@@
 	(symbol
 		(lib_id "Diode:BAT54J")
-		(at 168.91 60.96 180)
+		(at 170.18 60.96 0)
 		(unit 1)
 		(exclude_from_sim no)
@@
 		(fields_autoplaced yes)
 		(property "Reference" "D5"
-			(at 169.2275 54.61 0)
+			(at 169.8625 54.61 0)
 			(effects
 				(font
@@
 		)
 		(property "Value" "BAT54J"
-			(at 169.2275 57.15 0)
+			(at 169.8625 57.15 0)
 			(effects
 				(font
@@
 		)
 		(property "Footprint" "Diode_SMD:D_SOD-323F"
-			(at 168.91 56.515 0)
+			(at 170.18 65.405 0)
 			(effects
 				(font
@@
 		)
 		(property "Datasheet" "https://assets.nexperia.com/documents/data-sheet/BAT54J.pdf"
-			(at 168.91 60.96 0)
+			(at 170.18 60.96 0)
 			(effects
 				(font
@@
 		)
 		(property "Description" "30V 200mA Schottky diode, SOD-323F"
-			(at 168.91 60.96 0)
+			(at 170.18 60.96 0)
 			(effects
 				(font
