File: v0.1/sheets/camera.kicad_sch (KiCad schematic)
At the start: 4 parts

Commit message: [HW] [PCB] v.01 phase #3
Parts:
- added SCL1, SDA1: TestPoint, TestPoint:TestPoint_Pad_D1.0mm, symbol Connector:TestPoint
Connections:
- net DVP_SCL: now also SCL1.1
- net DVP_SDA: now also SDA1.1
Changed lines of the file:
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@@
 	(generator_version "9.0")
 	(paper "A4")
+	(junction
+		(at 160.02 67.31)
+		(diameter 0)
+		(color 0 0 0 0)
+	)
+	(junction
+		(at 154.94 72.39)
+		(diameter 0)
+		(color 0 0 0 0)
+	)
 	(bus_entry
 		(at 113.03 87.63)
@@
 		)
 	)
+	(wire
+		(pts
+			(xy 154.94 72.39) (xy 163.83 72.39)
+		)
+		(stroke
+			(width 0)
+			(type default)
+		)
+	)
+	(wire
+		(pts
+			(xy 154.94 52.07) (xy 154.94 72.39)
+		)
+		(stroke
+			(width 0)
+			(type default)
+		)
+	)
 	(bus
 		(pts
@@
 	(wire
 		(pts
+			(xy 160.02 67.31) (xy 163.83 67.31)
+		)
+		(stroke
+			(width 0)
+			(type default)
+		)
+	)
+	(wire
+		(pts
 			(xy 151.13 80.01) (xy 163.83 80.01)
 		)
@@
 	(wire
 		(pts
+			(xy 160.02 52.07) (xy 160.02 67.31)
+		)
+		(stroke
+			(width 0)
+			(type default)
+		)
+	)
+	(wire
+		(pts
 			(xy 139.7 92.71) (xy 163.83 92.71)
 		)
@@
 	(wire
 		(pts
-			(xy 151.13 67.31) (xy 163.83 67.31)
+			(xy 151.13 67.31) (xy 160.02 67.31)
 		)
 		(stroke
@@
 	(wire
 		(pts
-			(xy 151.13 72.39) (xy 163.83 72.39)
+			(xy 151.13 72.39) (xy 154.94 72.39)
 		)
 		(stroke
@@
 		(dnp no)
 		(fields_autoplaced yes)
-		(property "Reference" "#PWR049"
+		(property "Reference" "#PWR063"
 			(at 172.72 137.16 0)
 			(effects
@@
 			(project "v0.1"
 				(path "/d5a88f92-aedf-4ebc-b36f-cbb4d57161cd/046093c5-fb2a-4e8d-992c-23a84ae75cd9"
-					(reference "#PWR049")
+					(reference "#PWR063")
 					(unit 1)
 				)
@@
 		(dnp no)
 		(fields_autoplaced yes)
-		(property "Reference" "#PWR048"
+		(property "Reference" "#PWR062"
 			(at 172.72 44.45 0)
 			(effects
@@
 			(project "v0.1"
 				(path "/d5a88f92-aedf-4ebc-b36f-cbb4d57161cd/046093c5-fb2a-4e8d-992c-23a84ae75cd9"
-					(reference "#PWR048")
+					(reference "#PWR062")
+					(unit 1)
+				)
+			)
+		)
+	)
+	(symbol
+		(lib_id "Connector:TestPoint")
+		(at 154.94 52.07 0)
+		(unit 1)
+		(exclude_from_sim no)
+		(in_bom yes)
+		(on_board yes)
+		(dnp no)
+		(property "Reference" "SCL1"
+			(at 152.908 45.974 0)
+			(effects
+				(font
+					(size 1.27 1.27)
+				)
+				(justify left)
+			)
+		)
+		(property "Value" "TestPoint"
+			(at 148.336 43.942 0)
+			(effects
+				(font
+					(size 1.27 1.27)
+				)
+				(justify left)
+			)
+		)
+		(property "Footprint" "TestPoint:TestPoint_Pad_D1.0mm"
+			(at 160.02 52.07 0)
+			(effects
+				(font
+					(size 1.27 1.27)
+				)
+				(hide yes)
+			)
+		)
+		(property "Datasheet" "~"
+			(at 160.02 52.07 0)
+			(effects
+				(font
+					(size 1.27 1.27)
+				)
+				(hide yes)
+			)
+		)
+		(property "Description" "test point"
+			(at 154.94 52.07 0)
+			(effects
+				(font
+					(size 1.27 1.27)
+				)
+				(hide yes)
+			)
+		)
+		(pin "1"
+		)
+		(instances
+			(project "v0.1"
+				(path "/d5a88f92-aedf-4ebc-b36f-cbb4d57161cd/046093c5-fb2a-4e8d-992c-23a84ae75cd9"
+					(reference "SCL1")
+					(unit 1)
+				)
+			)
+		)
+	)
+	(symbol
+		(lib_id "Connector:TestPoint")
+		(at 160.02 52.07 0)
+		(unit 1)
+		(exclude_from_sim no)
+		(in_bom yes)
+		(on_board yes)
+		(dnp no)
+		(property "Reference" "SDA1"
+			(at 159.004 46.482 0)
+			(effects
+				(font
+					(size 1.27 1.27)
+				)
+				(justify left)
+			)
+		)
+		(property "Value" "TestPoint"
+			(at 158.242 43.942 0)
+			(effects
+				(font
+					(size 1.27 1.27)
+				)
+				(justify left)
+			)
+		)
+		(property "Footprint" "TestPoint:TestPoint_Pad_D1.0mm"
+			(at 165.1 52.07 0)
+			(effects
+				(font
+					(size 1.27 1.27)
+				)
+				(hide yes)
+			)
+		)
+		(property "Datasheet" "~"
+			(at 165.1 52.07 0)
+			(effects
+				(font
+					(size 1.27 1.27)
+				)
+				(hide yes)
+			)
+		)
+		(property "Description" "test point"
+			(at 160.02 52.07 0)
+			(effects
+				(font
+					(size 1.27 1.27)
+				)
+				(hide yes)
+			)
+		)
+		(pin "1"
+		)
+		(instances
+			(project ""
+				(path "/d5a88f92-aedf-4ebc-b36f-cbb4d57161cd/046093c5-fb2a-4e8d-992c-23a84ae75cd9"
+					(reference "SDA1")
 					(unit 1)
 				)
@@
 		)
 		(instances
-			(project "v0.1"
+			(project ""
 				(path "/d5a88f92-aedf-4ebc-b36f-cbb4d57161cd/046093c5-fb2a-4e8d-992c-23a84ae75cd9"
 					(reference "U11")
@@
 		(dnp no)
 		(fields_autoplaced yes)
-		(property "Reference" "#PWR046"
+		(property "Reference" "#PWR060"
 			(at 128.27 120.65 0)
 			(effects
@@
 			(project "v0.1"
 				(path "/d5a88f92-aedf-4ebc-b36f-cbb4d57161cd/046093c5-fb2a-4e8d-992c-23a84ae75cd9"
-					(reference "#PWR046")
+					(reference "#PWR060")
 					(unit 1)
 				)
@@
 		(dnp no)
 		(fields_autoplaced yes)
-		(property "Reference" "#PWR047"
+		(property "Reference" "#PWR061"
 			(at 144.78 97.79 0)
 			(effects
@@
 		)
 		(instances
-			(project "v0.1"
+			(project ""
 				(path "/d5a88f92-aedf-4ebc-b36f-cbb4d57161cd/046093c5-fb2a-4e8d-992c-23a84ae75cd9"
-					(reference "#PWR047")
+					(reference "#PWR061")
 					(unit 1)
 				)

Commit message: [HW] [PCB] v0.1_Y48 revision
Parts:
- SCL1, SDA1: now left out of the parts list
- U11: LCSC Part # (none) -> C9900012923
Changed lines of the file:
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@@
 		(unit 1)
 		(exclude_from_sim no)
-		(in_bom yes)
+		(in_bom no)
 		(on_board yes)
 		(dnp no)
@@
 		(unit 1)
 		(exclude_from_sim no)
-		(in_bom yes)
+		(in_bom no)
 		(on_board yes)
 		(dnp no)
@@
 			(at 168.91 91.44 0)
 			(effects
+				(font
+					(size 1.27 1.27)
+				)
+				(hide yes)
+			)
+		)
+		(property "LCSC Part #" "C9900012923"
+			(at 168.91 91.44 0)
+			(effects

Commit message: [HW] [PCB] revision v0.1_Y49
Parts:
- added TP23, TP24, TP25: TestPoint, TestPoint:TestPoint_Pad_D1.0mm, symbol Connector:TestPoint
- renumbered JP13 to JP12, JP14 to JP13, R21 to R17
Connections:
- net DVP_HSYNC: now also TP24.1
- net DVP_PCLK: now also TP25.1
- net DVP_VSYNC: now also TP23.1
Other:
- moved on the sheet: SCL1, SDA1

Commit message: [HW] [PCB] PCB Revision 0.2_Y50; DK1
Parts:
- U11: footprint Grinreflex:FPC-SMD_24P-P0.50_SHOU-HAN_CTSJ-H2.0 -> Grinreflex:FFC-SMD_24P-P0.50_FH34SRJ-24S-0.5SH
- renumbered JP12 to JP11, JP13 to JP12
Changed lines of the file:
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@@
 		(on_board yes)
 		(dnp no)
-		(property "Reference" "JP13"
+		(property "Reference" "JP12"
 			(at 148.082 121.92 0)
 			(effects
@@
 			(project "v0.1"
 				(path "/d5a88f92-aedf-4ebc-b36f-cbb4d57161cd/046093c5-fb2a-4e8d-992c-23a84ae75cd9"
-					(reference "JP13")
+					(reference "JP12")
 					(unit 1)
 				)
@@
 			)
 		)
-		(property "Footprint" "Grinreflex:FPC-SMD_24P-P0.50_SHOU-HAN_CTSJ-H2.0"
+		(property "Footprint" "Grinreflex:FFC-SMD_24P-P0.50_FH34SRJ-24S-0.5SH"
 			(at 168.91 91.44 0)
 			(effects
@@
 		(on_board yes)
 		(dnp no)
-		(property "Reference" "JP12"
+		(property "Reference" "JP11"
 			(at 148.082 119.38 0)
 			(effects
@@
 			(project "v0.1"
 				(path "/d5a88f92-aedf-4ebc-b36f-cbb4d57161cd/046093c5-fb2a-4e8d-992c-23a84ae75cd9"
-					(reference "JP12")
-					(unit 1)
-				)
+					(reference "JP11")
+					(unit 1)
+				)
