File: v0.1/sheets/clock_reset.kicad_sch (KiCad schematic)
At the start: 8 parts, among them X1 32.768kHz, X2 16MHz

Commit message: [HW] [PCB] v0.1_Y48 revision
Parts:
- SW1: LCSC Part # (none) -> C221791
- X1: LCSC Part # (none) -> C145140
- X2: LCSC Part # (none) -> C193746
Changed lines of the file:
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@@
+			)
+		)
+		(property "LCSC Part #" "C221791"
+			(at 125.73 96.52 90)
+			(effects
+				(font
+					(size 1.27 1.27)
+				)
+				(hide yes)
 			)
 		)
@@
 			)
 		)
+		(property "LCSC Part #" "C145140"
+			(at 72.39 125.73 0)
+			(effects
+				(font
+					(size 1.27 1.27)
+				)
+				(hide yes)
+			)
+		)
 		(pin "1"
 		)
@@
 			(at 73.66 97.79 0)
 			(effects
+				(font
+					(size 1.27 1.27)
+				)
+				(hide yes)
+			)
+		)
+		(property "LCSC Part #" "C193746"
+			(at 73.66 97.79 0)
+			(effects

Commit message: [HW] [PCB] revision v0.1_Y49
Parts:
- added C54: 100nf, Capacitor_SMD:C_0603_1608Metric, symbol Device:C_Small
- added R18: 100k, Resistor_SMD:R_0603_1608Metric, symbol Device:R_Small
- added R19: 1.5k, Resistor_SMD:R_0603_1608Metric, symbol Device:R_Small
- added U12: ~, Grinreflex:SOT-23-3_L2.9-W1.6-P1.90-LS2.8-BR, symbol Grinreflex:MAX809TEUR+T
- renumbered C38 to C50, C39 to C51, C40 to C52, C41 to C53, C42 to C55
Connections:
- net GND: now also C54.1, R18.2, U12.1 (GND)
- net RESET: now also R19.2
- new net: R18.1, R19.1, U12.2 (RESET)
- new net VCC: C54.2, U12.3 (VCC)
Other:
- moved on the sheet: C55, SW1

Commit message: [HW] [PCB] PCB Revision 0.2_Y50; DK1
Parts:
- added R20: 100k, Resistor_SMD:R_0402_1005Metric, symbol Device:R_Small
- C50, C51, C52, C53, C54: footprint Capacitor_SMD:C_0603_1608Metric -> Capacitor_SMD:C_0402_1005Metric
- R18, R19: footprint Resistor_SMD:R_0603_1608Metric -> Resistor_SMD:R_0402_1005Metric
Connections:
- net RESET: now also R20.2
- net VCC: now also R20.1
Changed lines of the file:
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@@
+	(wire
+		(pts
+			(xy 153.67 86.36) (xy 153.67 91.44)
+		)
+		(stroke
+			(width 0)
+			(type default)
+		)
+	)
 	(wire
 		(pts
@@
 		(pts
 			(xy 171.45 91.44) (xy 171.45 96.52)
+		)
+		(stroke
+			(width 0)
+			(type default)
+		)
+	)
+	(wire
+		(pts
+			(xy 153.67 73.66) (xy 153.67 81.28)
 		)
 		(stroke
@@
 		(shape input)
 		(at 66.04 125.73 90)
+		(effects
+			(font
+				(size 1.27 1.27)
+			)
+			(justify left)
+		)
+	)
+	(hierarchical_label "VCC"
+		(shape input)
+		(at 153.67 73.66 90)
 		(effects
 			(font
@@
 			)
 		)
-		(property "Footprint" "Capacitor_SMD:C_0603_1608Metric"
+		(property "Footprint" "Capacitor_SMD:C_0402_1005Metric"
 			(at 86.36 95.25 0)
 			(effects
@@
 			)
 		)
-		(property "Footprint" "Resistor_SMD:R_0603_1608Metric"
+		(property "Footprint" "Resistor_SMD:R_0402_1005Metric"
 			(at 135.89 97.79 0)
 			(effects
@@
 			)
 		)
-		(property "Footprint" "Capacitor_SMD:C_0603_1608Metric"
+		(property "Footprint" "Capacitor_SMD:C_0402_1005Metric"
 			(at 66.04 130.81 0)
 			(effects
@@
 			)
 		)
-		(property "Footprint" "Capacitor_SMD:C_0603_1608Metric"
+		(property "Footprint" "Capacitor_SMD:C_0402_1005Metric"
 			(at 60.96 100.33 0)
 			(effects
@@
 			)
 		)
-		(property "Footprint" "Resistor_SMD:R_0603_1608Metric"
+		(property "Footprint" "Resistor_SMD:R_0402_1005Metric"
 			(at 146.05 91.44 0)
 			(effects
@@
 			)
 		)
-		(property "Footprint" "Capacitor_SMD:C_0603_1608Metric"
+		(property "Footprint" "Capacitor_SMD:C_0402_1005Metric"
 			(at 80.01 130.81 0)
 			(effects
@@
 			)
 		)
-		(property "Footprint" "Capacitor_SMD:C_0603_1608Metric"
+		(property "Footprint" "Capacitor_SMD:C_0402_1005Metric"
 			(at 130.81 81.28 0)
 			(effects
@@
 					(unit 1)
 				)
+			)
+		)
+	)
+	(symbol
+		(lib_id "Device:R_Small")
+		(at 153.67 83.82 0)
+		(unit 1)
+		(exclude_from_sim no)
+		(in_bom yes)
+		(on_board yes)
+		(dnp no)
+		(fields_autoplaced yes)
+		(property "Reference" "R20"
+			(at 156.21 82.5499 0)
+			(effects
+				(font
+					(size 1.016 1.016)
+				)
+				(justify left)
+			)
+		)
+		(property "Value" "100k"
+			(at 156.21 85.0899 0)
+			(effects
+				(font
+					(size 1.27 1.27)
+				)
+				(justify left)
+			)
+		)
+		(property "Footprint" "Resistor_SMD:R_0402_1005Metric"
+			(at 153.67 83.82 0)
+			(effects
+				(font
+					(size 1.27 1.27)
+				)
+				(hide yes)
+			)
+		)
+		(property "Datasheet" "~"
+			(at 153.67 83.82 0)
+			(effects
+				(font
+					(size 1.27 1.27)
+				)
+				(hide yes)
+			)
+		)
+		(property "Description" "Resistor, small symbol"
+			(at 153.67 83.82 0)
+			(effects
+				(font
+					(size 1.27 1.27)
+				)
+				(hide yes)
+			)
+		)
+		(pin "1"
+		)
+		(pin "2"
+		)
+		(instances
+			(project "v0.1"
+				(path "/d5a88f92-aedf-4ebc-b36f-cbb4d57161cd/71a855a2-7e54-4076-a3fd-ce99cd30d9cf"
+					(reference "R20")
+					(unit 1)
+				)
