File: v0.1/sheets/flash.kicad_sch (KiCad schematic)
At the start: 17 parts, among them U9 MX66LM1G45G

Commit message: [HW] [PCB] v.01 phase #3
Parts:
- renumbered TP4 to TP10, TP6 to TP11, TP7 to TP12, TP8 to TP13, TP9 to TP14, TP10 to TP15, TP11 to TP16, TP12 to TP17, TP13 to TP18, TP2 to TP8, TP3 to TP9

Commit message: [HW] [PCB] v0.1_Y48 revision
Parts:
- TP10, TP11, TP12, TP13, TP14, TP15, TP16, TP17, TP18, TP8, TP9: now left out of the parts list
- U9: footprint Package_SO:SOP-16_3.9x9.9mm_P1.27mm -> Package_SO:SOIC-16W_7.5x10.3mm_P1.27mm
Changed lines of the file:
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@@
 		(unit 1)
 		(exclude_from_sim no)
-		(in_bom yes)
+		(in_bom no)
 		(on_board yes)
 		(dnp no)
@@
 		(unit 1)
 		(exclude_from_sim no)
-		(in_bom yes)
+		(in_bom no)
 		(on_board yes)
 		(dnp no)
@@
 		(unit 1)
 		(exclude_from_sim no)
-		(in_bom yes)
+		(in_bom no)
 		(on_board yes)
 		(dnp no)
@@
 		(unit 1)
 		(exclude_from_sim no)
-		(in_bom yes)
+		(in_bom no)
 		(on_board yes)
 		(dnp no)
@@
 		(unit 1)
 		(exclude_from_sim no)
-		(in_bom yes)
+		(in_bom no)
 		(on_board yes)
 		(dnp no)
@@
 			)
 		)
-		(property "Footprint" "Package_SO:SOP-16_3.9x9.9mm_P1.27mm"
+		(property "Footprint" "Package_SO:SOIC-16W_7.5x10.3mm_P1.27mm"
 			(at 152.4 81.28 0)
 			(effects
@@
 		(unit 1)
 		(exclude_from_sim no)
-		(in_bom yes)
+		(in_bom no)
 		(on_board yes)
 		(dnp no)
@@
 		(unit 1)
 		(exclude_from_sim no)
-		(in_bom yes)
+		(in_bom no)
 		(on_board yes)
 		(dnp no)
@@
 		(unit 1)
 		(exclude_from_sim no)
-		(in_bom yes)
+		(in_bom no)
 		(on_board yes)
 		(dnp no)
@@
 		(unit 1)
 		(exclude_from_sim no)
-		(in_bom yes)
+		(in_bom no)
 		(on_board yes)
 		(dnp no)
@@
 		(unit 1)
 		(exclude_from_sim no)
-		(in_bom yes)
+		(in_bom no)
 		(on_board yes)
 		(dnp no)
@@
 		(unit 1)
 		(exclude_from_sim no)
-		(in_bom yes)
-		(on_board yes)
-		(dnp no)
+		(in_bom no)
+		(on_board yes)
+		(dnp no)

Commit message: [HW] [PCB] revision v0.1_Y49
Parts:
- renumbered R19 to R15
Changed lines of the file:
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@@
 		(on_board yes)
 		(dnp no)
-		(property "Reference" "R19"
+		(property "Reference" "R15"
 			(at 118.11 80.518 0)
 			(effects
@@
 			(project "v0.1"
 				(path "/d5a88f92-aedf-4ebc-b36f-cbb4d57161cd/1214c110-4dbe-46ce-a863-01281192e9ea"
-					(reference "R19")
+					(reference "R15")
 					(unit 1)
 				)
