File: v1.0/v1.0.kicad_pcb (KiCad board)
At the start: 4 copper layers, 35 x 44 mm, 73 parts, among them IC1 STM32U5G7VJT6Q, J1 Conn_01x05_Pin, J3 Conn_01x02_Pin, J4 Conn_01x02_Pin, J5 Conn_01x02_Pin, J6 Conn_01x02_Pin, J7 Conn_01x02_Pin, U6 XC6206P152MR, U7 XC6206P282MR, U8 SY8088AAC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

Commit message: Revision V2.0 finalized
Parts:
- added C34: 100nF, Capacitor_SMD:C_0402_1005Metric, F.Cu at (111.6, 108.5)
- added C38: 100nF, Capacitor_SMD:C_0402_1005Metric, B.Cu at (107.2, 110.4)
- added C39: 100nF, Capacitor_SMD:C_0402_1005Metric, F.Cu at (92.2, 104.2)
- added C40: 100nF, Capacitor_SMD:C_0402_1005Metric, F.Cu at (90.5, 118.1)
- added C41: 100nF, Capacitor_SMD:C_0402_1005Metric, F.Cu at (109.4, 121.3)
- moved C22 3.26 mm to (115.5, 110.9), turned to 90 degrees
- moved R11 2.52 mm to (110.2, 95.7), turned to 90 degrees
- moved R12 1.22 mm to (107.9, 99.4)
- moved R15 0.61 mm to (115.5, 94.0), turned to 90 degrees
Routing:
- net /MCU/I2C2_SDA: track 38.6 -> 56.0 mm
- net +3V3: track 83.8 -> 95.1 mm
- net GND: track 74.5 -> 69.0 mm, vias 40 -> 118
- net /MCU/SWDIO: track 6.63 -> 11.8 mm
- net /MCU/RCC_OSC_OUT: track 5.46 -> 7.46 mm
- net /camera/AVDD-2V8: track 14.2 -> 15.0 mm
- net /MCU/SPI2_MISO: track 14.4 -> 14.9 mm
Other:
- board text added: "100nf"
