File: v2.0/v2.0/v2.0.kicad_sch (KiCad schematic)
At the start: 13 parts, among them J1 Conn_01x05_Pin, J2 Conn_01x02_Pin

Commit message: V2.0 Prototype Y61-9265739A
Parts:
- added J3: Conn_01x02_Pin, Connector_PinHeader_2.54mm:PinHeader_1x02_P2.54mm_Vertical, symbol Connector:Conn_01x02_Pin
Connections:
- net +5V: now also J3.1 (Pin_1)
- net GND: now also J3.2 (Pin_2)
- net VDD_3V3 renamed +3V3
- no-connect marks 1 -> 9

Commit message: backups, comments on schematic
Other:
- note added: "Issues with REV1.0 : * NOR IC "IO1" pin has "ringing", I pust shunt resistor, but maybe lowering frequency may solve it; impedance missmatch ? * Add BootRom Uart TX pin : PG10"
Changed lines of the file:
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@@
 	(generator_version "9.0")
 	(paper "A4")
+	(text "Issues with REV1.0 :\n* NOR IC \"IO1\" pin has \"ringing\", I pust shunt resistor,\nbut maybe lowering frequency may solve it;\nimpedance missmatch ?\n* Add BootRom Uart TX pin : PG10"
+		(exclude_from_sim no)
+		(at 34.29 132.334 0)
+		(effects
+			(font
+				(size 1.27 1.27)
+			)
+			(justify left)
+		)
+	)
 	(junction
 		(at 120.65 91.44)
