File: v2.0/v2.0/sheets/LCD.kicad_sch (KiCad schematic)
At the start: 6 parts

Commit message: V2.0 Prototype Y61-9265739A
Changed lines of the file:
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@@
-	(wire
-		(pts
-			(xy 132.08 78.74) (xy 132.08 88.9)
-		)
-		(stroke
-			(width 0)
-			(type default)
-		)
-	)
 	(wire
 		(pts
@@
 	(wire
 		(pts
+			(xy 132.08 78.74) (xy 132.08 88.9)
+		)
+		(stroke
+			(width 0)
+			(type default)
+		)
+	)
+	(wire
+		(pts
 			(xy 124.46 105.41) (xy 116.84 105.41)
 		)
@@
 	)
 	(label "LCD_CS"
-		(at 132.08 86.36 90)
+		(at 132.08 78.74 270)
 		(effects
 			(font
 				(size 1.27 1.27)
 			)
-			(justify left bottom)
+			(justify right bottom)
 		)
 	)
