File: v2.0/v2.0/sheets/MCU.kicad_sch (KiCad schematic)
At the start: 53 parts, among them IC1 STM32N657X0H3Q

Commit message: V2.0 Prototype Y61-9265739A
Parts:
- added JP7: SolderJumper_2_Open, Jumper:SolderJumper-2_P1.3mm_Open_RoundedPad1.0x1.5mm, symbol Jumper:SolderJumper_2_Open
- added TP10, TP11, TP12, TP13, TP14, TP15: TestPoint, TestPoint:TestPoint_Pad_D1.0mm, symbol Connector:TestPoint
- added U13: ~, Grinreflex:FFC-SMD_24P-P0.50_FH34SRJ-24S-0.5SH, symbol Grinreflex:FPC0.5-24P/上接抽拉
- IC1: footprint BGA264C80P17X17_1400X1400X100 -> v2.0:BGA264C80P17X17_1400X1400X100
Connections:
- net GND: now also U13.15, U13.16, U13.17, U13.18, U13.21, U13.22, U13.25, U13.26
- net I2C2_SDA: now also U13.2
- net VDDCORE: now also JP7.2 (B)
- net VDDIO: now also U13.23, U13.24
- net VDD_3V3: now also U13.19, U13.20
- net VFBSMPS: now also JP7.1 (A)
- net PD10: now reaches IC1.A13 (PD10)
- net PD10: now also U13.14
- net PD1: now reaches IC1.A14 (PD1)
- net PD1: now also U13.1
- net PE8: now reaches IC1.A15 (PE8)
- net PE8: now also U13.3
- net PE9: now reaches IC1.A16 (PE9)
- net PE9: now also U13.5
- net PD4: now reaches IC1.B15 (PD4)
- net PD4: now also U13.4
- net PE10: now reaches IC1.B16 (PE10)
- net PE10: now also U13.6
- net PB14: now reaches IC1.B17 (PB14)
- net PB14: now also U13.8
- net PB2: now reaches IC1.C16 (PB2)
- net PB2: now also U13.7
- net PD13: now reaches IC1.C17 (PD13)
- net PD13: now also U13.9
- net PB8: now reaches IC1.D16 (PB8)
- net PB8: now also U13.10
- net PB15: now reaches IC1.D17 (PB15)
- net PB15: now also U13.11
- net PE0: now reaches IC1.F16 (PE0)
- net PE0: now also U13.13
- net PE1: now reaches IC1.F17 (PE1)
- net PE1: now also U13.12
- net at IC1.T1 (PF12): now also TP15.1
- net at IC1.T12 (PB4): now also TP14.1
- net at IC1.U11 (PB10): now also TP13.1
- net at IC1.U12 (PB5): now also TP12.1
- net at IC1.U13 (PG11): now also TP11.1
- net at IC1.U14 (PA4): now also TP10.1
- no-connect marks 2 -> 118
Other:
- note added: "Switch smps -> external vddcore"
