File: v2.0/v2.0/sheets/power.kicad_sch (KiCad schematic)
At the start: 47 parts, among them U4 TPS62088YFP

Commit message: V2.0 Prototype Y61-9265739A
Parts:
- added TP9: TestPoint, TestPoint:TestPoint_Pad_D1.0mm, symbol Connector:TestPoint
Connections:
- net PWR_ON: now also TP9.1
Changed lines of the file:
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@@
 	)
 	(junction
+		(at 30.48 71.12)
+		(diameter 0)
+		(color 0 0 0 0)
+	)
+	(junction
 		(at 58.42 236.22)
 		(diameter 0)
@@
 	(wire
 		(pts
+			(xy 30.48 71.12) (xy 34.29 71.12)
+		)
+		(stroke
+			(width 0)
+			(type default)
+		)
+	)
+	(wire
+		(pts
 			(xy 245.11 113.03) (xy 247.65 113.03)
 		)
@@
 	(wire
 		(pts
+			(xy 30.48 64.77) (xy 30.48 71.12)
+		)
+		(stroke
+			(width 0)
+			(type default)
+		)
+	)
+	(wire
+		(pts
 			(xy 295.91 77.47) (xy 295.91 81.28)
 		)
@@
 	(wire
 		(pts
-			(xy 19.05 71.12) (xy 34.29 71.12)
+			(xy 19.05 71.12) (xy 30.48 71.12)
 		)
 		(stroke
@@
 			"AAAAAAAAAAAAAAAAAAAAAAAAAAAAAAAAAAAAAAAAAAAAAAAAAAAAAAAAAAAAAAAAAAAAAAAAAAAA"
 			"AAAAAAAAAAAAAAAAAAAAAAAAAAAAAAAAAAAAAAAAAAAAAAAAAAAAAAAAAAAAAAAAAAAAAAAAAAAA"
-			"AAAAAAAAAAAAAAAAAAAAAAAAAAAAAAAAAAAAAAAAAAAAAAAAAAAAAAAAAAAAAAAAAAAAAA=="
+			"AAAAAAAAAAAAAAAAAAAAAAAAAAAAAAAAAAAAAAAAAAAAAAAAAAAAAAAAAAAAAAAAAAAAADN8XgAA"
+			"8FlJNHxeAABwm7M0fF4AACBFZzV8XgAAsGmKNXxeAAAgAc9bLHEAAIB/jTR8XgAA4CFvNXxeAADw"
+			"v+EzfF4AAJDcbTR8XgAAUMuwNHxeAABwhHk1fF4AADBJUjR8XgAAAOKzNHxeAABQRmc1fF4AAECG"
+			"ijV8XgAAAAAAAAAAAACAgI00fF4AAGAjbzV8XgAA0MDhM3xeAABA3m00fF4AAGDRsDR8XgAAELt6"
+			"NXxeAAAQnlI0fF4AAND2szR8XgAAEEdnNXxeAACwh4o1fF4AAMD0DTV8XgAAoIGNNHxeAACgI281"
+			"fF4AANDB4TN8XgAA0N1tNHxeAACw1rA0fF4AAODqejV8XgAAoJ5SNHxeAABgdrQ0fF4AAPBHZzV8"
+			"XgAAUIeKNXxeAABg9Q01fF4AAOCCjTR8XgAAQDpvNXxeAADwwuEzfF4AAPDgbTR8XgAAYNiwNHxe"
+			"AAAgfnc1fF4AAHD41jN8XgAA0I+0NHxeAADwSGc1fF4AAOCOijV8XgAA/6XO0nleAAAwgo00fF4A"
+			"AOA5bzV8XgAAMMThM3xeAADw4W00fF4AAPDXsDR8XgAAQAR4NXxeAAAAoFI0fF4AAEAiZjR8XgAA"
+			"gEtnNXxeAADwj4o1fF4AAMDxDTV8XgAAYISNNHxeAACwPm81fF4AAIDD4TN8XgAAEONtNHxeAACQ"
+			"2rA0fF4AAPAEeDV8XgAA8IJSNHxeAADQO2Y0fF4AAFBMZzV8XgAAoJOKNXxeAAAAAAAAAAAAAACG"
+			"jTR8XgAAwD9vNXxeAACwxeEzfF4AACDpbTR8XgAAkNuwNHxeAADQBXg1fF4AACChUjR8XgAAUEZo"
+			"NHxeAADARGc1fF4AAAAAAAAAAAAAAAAAAAAAAADwhI00fF4AAMBCbzV8XgAAUMfhM3xeAABw7m00"
+			"fF4AALDcsDR8XgAA0AZ4NXxeAAAAolI0fF4AAHBgaDR8XgAAsE9nNXxeAAAQmYo1fF4AAP////8A"
+			"AAAAgIWNNHxeAABwRG81fF4AAEDG4TN8XgAA8O9tNHxeAADA5rA0fF4AAGCzdDV8XgAAAKNSNHxe"
+			"AADgiw41fF4AAJBQZzV8XgAAgJyKNXxeAAAgO+DJLHEAAMCFjTR8XgAAQEdvNXxeAADQxuEzfF4A"
+			"AIDvbTR8XgAAUOewNHxeAACgtHQ1fF4AACCkUjR8XgAA4JIONXxeAAAAU2c1fF4AAGCdijV8XgAA"
+			"YmlhcwAAAAAwe400fF4AAHBIbzV8XgAAEMfhM3xeAACA8m00fF4AAPDosDR8XgAAsKh0NXxeAABg"
+			"pVI0fF4AAOAYDzV8XgAAAFRnNXxeAABAoYo1fF4AAAAAAAAAAAAAkIaNNHxeAAAwSW81fA=="
 		)
 	)
@@
 			"AAAAAAAAAAAAAAAAAAAAAAAAAAAAAAAAAAAAAAAAAAAAAAAAAAAAAAAAAAAAAAAAAAAAAAAAAAAA"
 			"AAAAAAAAAAAAAAAAAAAAAAAAAAAAAAAAAAAAAAAAAAAAAAAAAAAAAAAAAAAAAAAAAAAAAAAAAAAA"
+			"AAAAAAAAAAAAAAAAAAAAAAAAAAAAAAAAAAAAAAAAAAAAAAAAAAAAAAAAAAAAAAAAAAAAAAAAAAAA"
+			"AAAAAAAAAAAAAAAAAAAAAAAAAAAAAAAAAAAAAAAAAAAAAAAAAAAAAAAAAAAAAAAAAAAAAAAAAAAA"
+			"AAAAAAAAAAAAAAAAAAAAAAAAAAAAAAAAAAAAAAAAAAAAAAAAAAAAAAAAAAAAAAAAAAAAAAAAAAAA"
+			"AAAAAAAAAAAAAAAAAAAAAAAAAAAAAAAAAAAAAAAAAAAAAAAAAAAAAAAAAAAAAAAAAAAAAAAAAAAA"
+			"AAAAAAAAAAAAAAAAAAAAAAAAAAAAAAAAAAAAAAAAAAAAAAAAAAAAAAAAAAAAAAAAAAAAAAAAAAAA"
+			"AAAAAAAAAAAAAAAAAAAAAAAAAAAAAAAAAAAAAAAAAAAAAAAAAAAAAAAAAAAAAAAAAAAAAAAAAAAA"
+			"AAAAAAAAAAAAAAAAAAAAAAAAAAAAAAAAAAAAAAAAAAAAAAAAAAAAAAAAAAAAAAAAAAAAAAAAAAAA"
+			"AAAAAAAAAAAAAAAAAAAAAAAAAAAAAAAAAAAAAAAAAAAAAAAAAAAAAAAAAAAAAAAAAAAAAAAAAAAA"
+			"AAAAAAAAAAAAAAAAAAAAAAAAAAAAAAAAAAAAAAAAAAAAAAAAAAAAAAAAAAAAAAAAAAAAAAAAAAAA"
+			"AAAAAAAAAAAAAAAAAAAAAAAAAAAAAAAAAAAAAAAAAAAAAAAAAAAAAAAAAAAAAAAAAAAAAAAAAAAA"
+			"AAAAAAAAAAAAAAAAAAAAAAAAAAAAAAAAAAAAAAAAAAAAAAAAAAAAAAAAAAAAAAAAAAAAAAAAAAAA"
+			"AAAAAAAAAAAAAAAAAAAAAAAAAAAAAAAAAAAAAAAAAAAAAAAAAAAAAAAAAAAAAAAAAAAAAAAAAAAA"
+			"AAAAAAAAAAAAAAAAAAAAAAAAAAAAAAAAAAAAAAAAAAAAAAAAAAAAAAAAAAAAAAAAAAAAAAAAAAAA"
+			"AAAAAAAAAAAAAAAAAAAAAAAAAAAAAAAAAAAAAAAAAAAAAAAAAAAAAAAAAAAAAAAAAAAAAAAAAAAA"
+			"AAAAAAAAAAAAAAAAAAAAAAAAAAAAAAAAAAAAAAAAAAAAAAAAAAAAAAAAAAAAAAAAAAAAAAAAAAAA"
+			"AAAAAAAAAAAAAAAAAAAAAAAAAAAAAAAAAAAAAAAAAAAAAAAAAAAAAAAAAAAAAAAAAAAAAAAAAAAA"
+			"AAAAAAAAAAAAAAAAAAAAAAAAAAAAAAAAAAAAAAAAAAAAAAAAAAAAAAAAAAAAAAAAAAAAAAAAAAAA"
+			"AAAAAAAAAAAAAAAAAAAAAAAAAAAAAAAAAAAAAAAAAAAAAAAAAAAAAAAAAAAAAAAAAAAAAAAAAAAA"
 			"AAAAAAAAAAAAAA=="
 		)
@@
 					(unit 1)
 				)
+			)
+		)
+	)
+	(symbol
+		(lib_id "Connector:TestPoint")
+		(at 30.48 64.77 0)
+		(unit 1)
+		(exclude_from_sim no)
+		(in_bom no)
+		(on_board yes)
+		(dnp no)
+		(fields_autoplaced yes)
+		(property "Reference" "TP9"
+			(at 33.02 60.1979 0)
+			(effects
+				(font
+					(size 1.27 1.27)
+				)
+				(justify left)
+			)
+		)
+		(property "Value" "TestPoint"
+			(at 33.02 62.7379 0)
+			(effects
+				(font
+					(size 1.27 1.27)
+				)
+				(justify left)
+			)
+		)
+		(property "Footprint" "TestPoint:TestPoint_Pad_D1.0mm"
+			(at 35.56 64.77 0)
+			(effects
+				(font
+					(size 1.27 1.27)
+				)
+				(hide yes)
+			)
+		)
+		(property "Datasheet" "~"
+			(at 35.56 64.77 0)
+			(effects
+				(font
+					(size 1.27 1.27)
+				)
+				(hide yes)
+			)
+		)
+		(property "Description" "test point"
+			(at 30.48 64.77 0)
+			(effects
+				(font
+					(size 1.27 1.27)
+				)
+				(hide yes)
+			)
+		)
+		(pin "1"
+		)
+		(instances
+			(project "v2.0"
+				(path "/358f9123-977b-4c66-b028-35bace4b0bfc/71e29154-573e-421d-a811-f0a5c599e99a"
+					(reference "TP9")
+					(unit 1)
+				)
